File: CPU.kicad_sch (KiCad schematic)
At the start: 147 parts, among them P1 Conn_02x36_Top_Bottom, P3 Conn_02x13_Top_Bottom, P4 Conn_02x13_Top_Bottom, P5 Conn_02x25_Counter_Clockwise, P6 Conn_02x25_Counter_Clockwise, P7_L12 Conn_02x07_Counter_Clockwise

Commit message: update netlist
Parts:
- R12: renamed from R1; value R -> 4.7k
- R13: renamed from R2; value R -> 4.7k
- renumbered CRYSTAL to CRYSTAL1

Commit message: rev5: more traces from back of card
Parts:
- added R14: 1k, symbol Device:R
- added R8: 47, symbol Device:R
- R2, R3: value R -> 550
- XTAL1: renamed from CRYSTAL1; value Crystal -> 5.000MHz
- renumbered P7_L12 to P7
Connections:
- net +5V: now also U_E7.16 (VCC)
- net GND: now also U_E7.4 (E1), U_E7.5 (E2), U_H14.8 (GND), U_J13.8 (GND)
- net MW.H_{0}: now also U_J6.3
- net MW.J_{6}: now also U_E7.2 (A1)
- net P4_12: now also U_C9.17 (D6), U_D9.14 (D5)
- net P4_13: now also U_D9.13 (D4)
- net P7_3: now also P7.3 (Pin_3)
- net P7_4: now also P7.4 (Pin_4)
- net TODO_B8_6: now reaches U_C7.2
- net TODO_B8_6: now also U_B8.6
- net at R4.3 (R2): now also P4.10 (Pin_10), U_M8.8 (I3a)
- net ~{FPC_P4_M8_12}: now reaches U_D8.10
- net ~{FPC_P4_M8_12}: now also U_D8.5, U_M8.12 (O3a)
- net at U_D8.8: now also U_D7.2 (~{S1})
- net at U_C10.11: now also U_B15.12 (D), U_B15.2 (D)
- net P7_1: now reaches P7.1 (Pin_1)
- net P7_10: now reaches P7.10 (Pin_10)
- net P7_11: now reaches P7.11 (Pin_11)
- net P7_12: now reaches P7.12 (Pin_12)
- net P7_13: now reaches P7.13 (Pin_13)
- net P7_14: now reaches P7.14 (Pin_14)
- net P7_2: now reaches P7.2 (Pin_2)
- net P7_5: now reaches P7.5 (Pin_5)
- net P7_6: now reaches P7.6 (Pin_6)
- net P7_7: now reaches P7.7 (Pin_7)
- net P7_8: now reaches P7.8 (Pin_8)
- net P7_9: now reaches P7.9 (Pin_9)
- net TODO_D7_11_M6_16: now reaches U_D7.11 (CP)
- net TODO_D7_11_M6_16: now also U_D7.5 (CP)
- net at U_D7.13 (~{S1}): now also U_D8.6
- net at U_D7.15 (M): now also U_D7.1 (M), R14.1
- net at U_L13.1 (~{R}): now also U_J13.1 (Ea), U_J13.15 (Eb)
- net at U_J13.10 (I0b): now also U_J12.11 (I1b)
- net Sys.E_{57}: now reaches P1.57 (Pin_57), U_A8.1 (BUS0)
- net Sys.E_{55}: now reaches P1.55 (Pin_55), U_A8.12 (BUS2)
- net Sys.E_{54}: now reaches P1.54 (Pin_54), U_A8.15 (BUS3)
- net Sys.E_{56}: now reaches P1.56 (Pin_56), U_A8.4 (BUS1)
- net TODO_F11_12_E11_13: now reaches U_F11.12 (Q7)
- net TODO_F11_12_E11_13: now also U_E11.13
- net F11_EN: now reaches U_F11.14 (E)
- net F11_EN: now also U_K11.12 (O3)
- net ~{F11_Clear}: now reaches U_F11.15 (Clr)
- net ~{F11_Clear}: now also U_D4.5 (Q1)
- net M8_I0b: now reaches U_F11.9 (Q4)
- net M8_I0b: now also U_M8.11 (I0b)
- net at U_K6.1, U_K6.5, U_K6.9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: now also R8.2
- net at U_K10.1: now also U_J9.14 (D5); no longer U_J9.15 (Q5)
- net at U_K10.2: now also U_J9.15 (Q5); no longer U_J9.14 (D5)
- net at U_M13.4 (Q0): now also U_M8.13 (I1b)
- net at U_M13.5 (Q1): now also U_M8.15 (I2b)
- net F14C_b: now reaches U_M13.6 (Q2)
- net F14C_b: now also U_F14.10
- net at U_D12.5: now also U_C10.8
- net at U_D12.6: now also U_D7.3 (~{S2})
- net at P4.2 (Pin_2): now also U_M8.9 (O0b)
- net at P4.3 (Pin_3): now also U_M8.7 (O1b)
- net at P4.4 (Pin_4): now also U_M8.5 (O2b)
- net at P4.6 (Pin_6): now also U_M8.16 (O1a), U_M8.3 (O3b)
- net Sys.E58: now reaches P1.58 (Pin_58)
- net Sys.E58: now also U_C8.2
- net at U_C9.13 (D4): now also U_D9.3 (D0)
- net ~{D9_EN}: now reaches U_D9.1 (~{E})
- net ~{D9_EN}: now also U_E6.12 (O3)
- net at U_F14.8: now also U_F13.14 (D5)
- net F14C_a: now reaches U_F14.9
- net F14C_a: now also U_M9.9 (Q)
- net at U_M12.3 (D0): now also U_J12.9 (Zb)
- net at U_J12.3 (I3a), U_J9.5 (Q1): now also U_J12.5 (I1a)
- net K9p15_I5: now reaches U_F14.6
- net K9p15_I5: now also U_K9.14 (I5)
- net at U_K9.6 (~{Z}): now also R8.1
- no-connect marks 21 -> 22
Other:
- note added: "ALU HIGH"
- note added: "ALU LOW"
- moved on the sheet: P7, R4, R7, U_C10D, U_C10E, U_C7A, U_C8A, U_D12B, U_D7A, U_D7B, U_D8B, U_F14A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

Commit message: clock control and misc logic
Parts:
- added BODGE1: Jumper_2_Bridged, symbol Jumper:Jumper_2_Bridged
- added R17, R9: 1k, symbol Device:R
- renumbered P4 to P2
Connections:
- net A1_10-D7_7 is gone; now on net ~{A1B_SET}: U_A1.10 (~{S}), U_D7.7 (~{Y})
- net SW_R is gone; now on net P7_13: DSW1.5, R7.3 (R2), U_M7.2 (I0a)
- net +5V: now also R6.1, R17.2, R9.2; no longer R6.2
- net A1_8-B11_4: now also U_B11.5, U_F12.3 (C)
- net P7_1: now also R6.2, U_L11.1 (S)
- net P7_13: now also BODGE1.1 (A)
- net P7_2: now also U_L11.5 (I0b), U_L14.4
- net P7_4: now also U_L10.12 (D), U_M10.11; no longer R3.1, U_L11.3 (I1a), U_M10.6, XTAL1.1
- net P7_5: now also U_L10.10 (~{S}), U_L10.4 (~{S}), R17.1
- net P7_8: now also U_L11.14 (I0d)
- net ~{ClockB_{1}}: now also U_F12.11 (C), U_F13.9 (Cp)
- net ~{M7_OEb}: now also U_M12.2 (Q0), U_M14.1 (OEa)
- net ~{A1_E15_F12_RESET}: now reaches U_F12.1 (~{R})
- net ~{A1_E15_F12_RESET}: now also U_A1.1 (~{R}), U_A1.13 (~{R}), U_D4.15 (Q5), U_E15.1 (~{R}), U_E15.13 (~{R})
- net ~{A1B_SET}: now reaches U_F12.4 (~{S})
- net M10C_b: now reaches U_F12.5 (Q)
- net M10C_b: now also U_M10.10
- net J11_IN_{0}_IN_{4}: now reaches U_F12.6 (~{Q})
- net J11_IN_{0}_IN_{4}: now also U_J11.15 (I4), U_J11.4 (I0)
- net F12B_D: now reaches U_C10.4, U_D6.3 (I1a)
- net F12B_D: now also U_F12.12 (D)
- net at U_M10.12: now also U_L10.2 (D), U_L10.9 (Q), U_L11.13 (I1d), BODGE1.2 (B)
- net TODO_M10_13: now reaches U_M10.13
- net TODO_M10_13: now also U_L11.6 (I1b)
- net ~{P7_2}: now reaches U_L14.6
- net ~{P7_2}: now also U_L11.11 (I0c)
- net FPC_P2_12: now reaches P2.12 (Pin_12), R4.5 (R4)
- net FPC_P2_12: now also U_M14.11 (I0b)
- net M10C_a: now reaches U_D8.12, U_D8.2, U_E11.5, U_E14.10, U_E8.11
- net M10C_a: now also U_D12.10, U_H12.1 (M), U_M10.9
- net at U_K13.1 (Ea): now also U_J13.1 (Ea), U_J13.15 (Eb), U_K13.15 (Eb)
- net at U_M14.13 (I1b): now also U_M13.11 (Q6)
- net at U_M14.15 (I2b): now also U_M13.9 (Q4)
- net at U_M14.17 (I3b): now also U_M14.5 (O2b)
- net at U_M14.4 (I1a), U_M15.4 (I1a): now also U_M12.4 (D1)
- net at P3.2 (Pin_2), U_M14.6 (I2a), U_M15.6 (I2a): now also U_J11.13 (I6), U_J11.2 (I2), U_M12.7 (Q2)
- net L13_~{K}: now reaches U_L13.3 (~{K})
- net L13_~{K}: now also U_D12.8
- net at U_L13.4 (C): now also U_L11.9 (Zc), U_M9.3 (C)
- net ~{L13A_SET}: now reaches U_L13.5 (~{S})
- net ~{L13A_SET}: now also U_K11.14 (O1)
- net at U_L13.7 (~{Q}): now also U_M8.4 (I1a)
- net D13_12_F9_25: now reaches U_D13.12 (O4)
- net D13_12_F9_25: now also U_F9.25 (D0), U_H14.9 (O4a)
- net D13_9_F7_25: now reaches U_D13.9 (O3)
- net D13_9_F7_25: now also U_F7.25 (D0)
- net at U_L10.1 (~{R}): now also U_L10.13 (~{R}), R9.1
- net at U_L10.6 (~{Q}): now also U_L11.10 (I1c)
- net ~{REGF.WE}: now reaches U_D14.20 (~{WE}), U_D15.20 (~{WE}), U_H13.8
- net at U_J11.5 (Z): now also U_M12.6 (D2)
- net P4_7: now reaches U_E12.3
- net at P2.8 (Pin_8): now also U_M8.18 (O0a)
- net TODO_J10_2_H6_11: now reaches U_H6.11 (I1b), U_H6.5 (I1a)
- net TODO_J10_2_H6_11: now also U_J10.2 (I2), U_J9.10 (Q3)
- net at U_M8.2 (I0a): now also U_M9.5 (Q)
- net at U_H12.14 (~{S2}): now also U_E14.8
- net TODO_M9_1: now reaches U_M9.1 (~{R})
- net TODO_M9_4: now reaches U_M9.4 (~{S})
- net TODO_C14_1_K5: now reaches U_C14.1 (S)
- net P10_8: now reaches U_K9.15 (I4)
- removed net P1_1: R6.1, U_L11.1 (S)
- net ~{ALTAddr_LD_LO} renamed ~{WorkAddr_LD_LO}
- net ~{ALTAddr_LOAD} renamed ~{WorkAddr_LD_HI}
- new net: R3.1, U_L11.3 (I1a), U_M10.6, XTAL1.1
- now unconnected: U_L13.1 (~{R})
- no-connect marks 22 -> 35
Other:
- note added: "EXT CLOCK OVERRIDE"
- note added: "Memory Address"
- note added: "SYSTEM CLOCK"
- note added: "Work Address High"
- note added: "Work Address Low"
- moved on the sheet: R2, R3, R6, R7, U_D12C, U_D13, U_E12B, U_E12C, U_E12D, U_E12E, U_E12F, U_E14B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

Commit message: candidates for C14 in
Connections:
- net E14A is gone; now on net TODO_E14_1_F11_5: U_D6.13 (I1d), U_D6.6 (I1b), U_E14.1
- net MW.J_{5}: now also U_E7.1 (A0)
- net ClockB_E8A: now reaches U_E14.13
- net ClockB_E8A: now also U_E8.1
- net TODO_D12_2_D8_8: now reaches U_D8.9
- net TODO_D12_2_D8_8: now also U_D12.2
- net TODO_H13_H11_D11: now reaches U_H13.13
- net TODO_C14_3: now reaches U_D10.11, U_D9.12 (Q4)
- net TODO_C14_3: now also U_C14.3 (I1a)
- net TODO_H13_6_K9-M9: now reaches U_H13.6
- net at U_E14.6: now also U_E15.11 (C)
- net TODO_C14_10: now reaches U_D10.9, U_D9.5 (Q1)
- net TODO_C14_10: now also U_C14.10 (I1c)
- net TODO_F14_F13: now reaches U_F14.4
- net TODO_F14_F13: now also U_F14.5
- net TODO_C14_15_GND: now reaches U_C14.15 (E)
- net A10_OE renamed TODO_E14_1_F11_5
Other:
- note added: "TODO"
- moved on the sheet: U_C10F, U_C11, U_C12, U_D11, U_E14C, U_F14B

Commit message: add labels, buses, fix area around B11,B12
Parts:
- added P4: Conn_02x08_Counter_Clockwise, symbol Connector_Generic:Conn_02x08_Counter_Clockwise
Connections:
- net P4_12 is gone; now on net DataF.D_{6}: U_C9.17 (D6), U_D9.14 (D5)
- net P4_13 is gone; now on net DataF.D_{7}: U_D9.13 (D4)
- net Address.A_{11}: now also U_B10.1 (A3)
- net DataA_{2}: now also U_B4.6 (I1b), U_B9.11 (D1), U_C9.6 (Q2)
- net DataF.D_{1}: now also P4.4 (Pin_4)
- net DataF.D_{6}: now also P4.12 (Pin_12)
- net DataF.D_{7}: now also U_C13.19 (Q7), U_C14.2 (I0a), U_C9.18 (D7), P4.13 (Pin_13)
- net MW.F_{0}: now also U_F9.5 (I_6)
- net MW.H_{1}: now also U_J13.1 (Ea), U_J13.15 (Eb), U_K13.1 (Ea), U_K13.15 (Eb)
- net SEQ.~{ZERO}: now also U_M13.15 (Clr)
- net TODO_B12_2: now also U_C10.11
- net B15_DAT: now reaches U_B11.12
- net B15_DAT: now also U_B15.12 (D), U_B15.2 (D)
- net at U_B11.13: now also U_B11.2
- net at U_B9.21 (A4): now also U_B10.21 (A4)
- net K7_OR_{0}: now reaches U_J13.7 (Za)
- net K7_OR_{0}: now also U_K7.12 (OR_{0})
- net K7_OR_{1}: now reaches U_J13.9 (Zb)
- net K7_OR_{1}: now also U_K7.10 (OR_{1})
- net at U_C4.6 (I1b): now also U_B10.11 (D1), U_C3.6 (I1b), U_C9.16 (Q6)
- net ALU.CARRY: now reaches U_F7.33 (Cn+4), U_H6.3 (I3a)
- net ~{C9_EN}: now reaches U_C9.1 (~{E})
- net ~{C9_EN}: now also U_E6.14 (O1)
- net TODO_M12_11_J10: now reaches U_M12.11 (D3)
- net Addr LOAD renamed MemAddr_LD_SWAP
- net P4_10 renamed DataF.D_{4}
- net DataF.D_{4}: now also P4.10 (Pin_10)
- net P4_11 renamed DataF.D_{5}
- net DataF.D_{5}: now also P4.11 (Pin_11)
- net P4_3 renamed DataF.D_{0}
- net DataF.D_{0}: now also P4.3 (Pin_3)
- net P4_5 renamed DataF.D_{2}
- net DataF.D_{2}: now also P4.5 (Pin_5)
- net P4_6 renamed DataF.D_{3}
- net DataF.D_{3}: now also P4.6 (Pin_6)
- net TODO_B1_1..2: no longer names the net of U_B2.2 (CP), U_B5.2 (CP), U_C2.2 (CP), U_C5.2 (CP), U_D6.9 (Zc)
- net ~{FPC_P4_M8_12} renamed ~{FPC_P2_M8_12}
- net ~{MUX_E_{0}E_{4}} renamed ~{SEL_E_{0}E_{4}}
- net ~{MUX_E_{10}} renamed ~{SEL_E_{10}}
- net ~{MUX_E_{11}} renamed ~{SEL_E_{11}}
- net ~{MUX_E_{12}} renamed ~{SEL_E_{12}}
- net ~{MUX_E_{13}} renamed ~{SEL_E_{13}}
- net ~{MUX_E_{1}E_{5}} renamed ~{SEL_E_{1}E_{5}}
- net ~{MUX_E_{2}E_{6}} renamed ~{SEL_E_{2}E_{6}}
- net ~{MUX_E_{3}E_{7}} renamed ~{SEL_E_{3}E_{7}}
- net ~{MUX_E_{8}} renamed ~{SEL_E_{8}}
- net ~{MUX_E_{9}} renamed ~{SEL_E_{9}}
Other:
- note added: "ALU Result"
- note added: "Condition Register"
- note added: "Frontpanel Drivers"
- note added: "Microcode Sequence Low > Hi"
- note added: "Page Table RAM"
- note added: "Register File RAM"
- note added: "Result Store"
- note added: "These may be the Address bus but traces for them are not visible"
- note added: "for the low order page RAM, the bits are stored and loaded in reverse of their pin order This is not visible to software"
- note added: "maybe B12_1 instead"
- moved on the sheet: U_C10E, U_D11, U_M12

Commit message: main clock-gen resolved
Connections:
- net LEVEL_LIMIT_15 is gone; now on net CLOCK_COUNT_15: U_A15.6, U_C15.7 (~{CEP})
- net MW.K_{4} is gone; now on net TODO_H6_2_K5_12: U_K5.12 (Q4)
- net TODO_M10_13 is gone; now on an unnamed net: U_L11.6 (I1b), U_M10.13
- net +5V: now also U_H11.6 (E3)
- net GND: now also U_H11.4 (E1), U_H11.5 (E2), U_L11.15 (E)
- net P7_2: now also U_L14.5
- net P7_3: now also U_L11.2 (I0a)
- net MainClockPhi2: now reaches U_L11.9 (Zc), U_L13.4 (C), U_M9.3 (C)
- net MainClockPhi2: now also U_H12.11 (CP), U_H12.5 (CP)
- net H12_~{S}: now reaches U_H12.13 (~{S1}), U_H12.2 (~{S1}), U_H12.3 (~{S2})
- net H12_~{S}: now also U_A3.12
- net TODO_B13_16_M13: now reaches U_B13.16 (~{CE2})
- net TODO_B13_16_M13: now also U_M13.7 (Q3)
- net MainClockPhi3: now reaches U_K12.6, U_L11.12 (Zd)
- net MainClockPhi1: now reaches U_L11.7 (Zb)
- net MainClockPhi1: now also U_C10.1
- net CLOCK_COUNT_15: now reaches U_A2.10, U_A2.9
- net TODO_H6_2_K5_12: now reaches U_F6.2 (S1), U_H6.2 (A1)
- no-connect marks 35 -> 38
Other:
- moved on the sheet: U_A2C, U_A3B, U_A3F

Commit message: bus control and condition pins
Connections:
- net TODO_D10_4_ROW_K is gone; now on net K9_In1: U_D10.4
- net TODO_D4_4 is gone; now on net Sys Reset: U_D4.14 (D5), U_D4.4 (D1), U_E7.6 (E3)
- net TODO_D6_2 is gone; now on net Addr_Clock: U_D6.11 (I0c), U_D6.2 (I0a)
- net TODO_F11_12_E11_13 is gone; now on net M8_I3b: U_E11.13, U_F11.12 (Q7)
- net TODO_H13_6_K9-M9 is gone; now on net K9_In7: U_H13.6
- net TODO_H13_H11_D11 is gone; now on an unnamed net: U_H13.13
- net ~{F11_Clear} is gone; now on net SEQ.~{ZERO}: U_D4.5 (Q1), U_F11.15 (Clr)
- net Addr U/D: now also U_F11.7 (Q3)
- net DataRDCLK: now also U_K11.7 (O7); no longer U_K11.10 (O5)
- net F13_D_{0}: no longer U_B15.3 (C)
- net GND: now also U_D6.15 (E)
- net P10_8: now also U_D12.1
- net ~{AND_SysE_{64}}: now reaches U_B11.13, U_B11.2
- net ~{AND_SysE_{64}}: now also U_F11.11 (Q6)
- net A13D_a: now reaches U_A13.12
- net A13D_a: now also U_F11.10 (Q5)
- net at U_K12.2: now also U_K12.3
- net K7_OR_{3}: now reaches U_K13.7 (Za)
- net K7_OR_{3}: now also U_K7.6 (OR_{3})
- net K7_OR_{2}: now reaches U_K13.9 (Zb)
- net K7_OR_{2}: now also U_K7.8 (OR_{2})
- net D7B_~{S2}: now reaches U_D7.14 (~{S2})
- net D7B_~{S2}: now also U_H11.14 (O1)
- net at U_A14.10, U_A15.2: now also U_A14.9
- net ~{PTRAM_WE}: now reaches U_B9.20 (~{WE})
- net ~{PTRAM_WE}: now also U_B10.20 (~{WE}), U_K11.10 (O5)
- net B12_~{F13_D_{0}}: now reaches U_F11.4 (Q0)
- net B12_~{F13_D_{0}}: now also U_B12.9
- net ~{AddrCount_EN}: now reaches U_F11.6 (Q2)
- net ~{AddrCount_EN}: now also U_D6.13 (I1d), U_D6.6 (I1b), U_E14.1
- net ClockA: now reaches U_E10.2, U_E11.3, U_H12.6 (Y)
- net K9_In0: now reaches U_F12.9 (Q)
- net K9_In0: now also U_K9.4 (I0)
- net ~{NibbleSwap_EN}: now reaches U_C11.10 (E2), U_C12.10 (E2), U_C12.9 (E1)
- net ~{NibbleSwap_EN}: now also U_C11.9 (E1), U_H11.7 (O7)
- net WorkAddr_Clock: now reaches U_D6.10 (I1c)
- net ~{WorkAddr_Count_EN}: now reaches U_D6.14 (I0d)
- net ~{WorkAddr_Count_EN}: now also U_H11.11 (O4)
- net ~{MemAddr_Count_EN}: now reaches U_D6.5 (I0b)
- net ~{MemAddr_Count_EN}: now also U_H11.10 (O5)
- net K9_In2: now reaches U_C13.2 (Q0)
- net K9_In2: now also U_K9.2 (I2)
- net D7A_~{S2}_Logic: now reaches U_C10.9
- net D7A_~{S2}_Logic: now also U_H11.13 (O2)
- net ~{DataRDLatch}: now reaches U_A11.1 (RLE), U_A12.1 (RLE), U_B12.6
- net M8_I3b: now reaches U_M8.17 (I3b)
- net Addr_Clock: now reaches U_H12.9 (~{Y})
- net at U_E8.13: now also U_B12.5
- net K9_In6: now reaches U_B15.6 (~{Q})
- net K9_In6: now also U_K9.13 (I6)
- net K9_In3: now reaches U_K9.1 (I3)
- net K9_In3: now also U_B12.3
- net K9_In7: now reaches U_K9.12 (I7)
- net K9_In1: now reaches U_K9.3 (I1)
- net K9p15_I5 renamed K9_In5
- net TODO_E14_1_F11_5 renamed A10_OE
- net A10_OE: no longer U_D6.13 (I1d), U_D6.6 (I1b), U_E14.1
- no-connect marks 38 -> 39
Other:
- note added: "Bus Control"
- note added: "Bus Control Function"
- note added: "Bus Control Register"
- moved on the sheet: P4, R14, U_B12B, U_B15A, U_B15B, U_C10F, U_D10A, U_D10B, U_D12C, U_E10A, U_E11A, U_E11B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

Commit message: microcode word renumber, layout changes
Connections:
- net K9_In2 is gone; now on net TODO_K9_D10_5: U_C13.2 (Q0), U_K9.2 (I2)
- net TODO_K9_D10_5: now reaches U_D10.3, U_D10.5
- net TODO_E12_4_B10: now reaches U_E12.4
- net TODO_K9_2or15or14_D10_6: now reaches U_D10.6
- net C13_EN renamed ~{C13_EN}
- net F13_D_{0}: no longer names the net of U_B12.8, U_F13.3 (D0)
- net K11MUX_{0} renamed MW.H6_{7}
- net K11MUX_{1} renamed MW.F5_{0}
- net MW.F5_{0}: no longer U_H13.12, U_J5.16 (Q6), U_K11.3 (A2)
- net MW.F_{0} renamed MW.B1_{0}
- net MW.F_{1} renamed MW.B1_{1}
- net MW.F_{2} renamed MW.B1_{2}
- net MW.F_{3} renamed MW.B1_{3}
- net MW.F_{7} renamed MW.B1_{7}
- net MW.H_{0} renamed MW.C2_{0}
- net MW.H_{1} renamed MW.C2_{1}
- net MW.H_{2} renamed MW.C2_{2}
- net MW.H_{3} renamed MW.C2_{3}
- net MW.H_{4} renamed MW.C2_{4}
- net MW.H_{5} renamed MW.C2_{5}
- net MW.H_{6} renamed MW.C2_{6}
- net MW.H_{7} renamed MW.C2_{7}
- net MW.J_{2} renamed MW.F5_{2}
- net MW.J_{3} renamed MW.F5_{3}
- net MW.J_{4} renamed MW.F5_{4}
- net MW.J_{5} renamed MW.F5_{5}
- net MW.J_{6} renamed MW.F5_{6}
- net MW.J_{7} renamed MW.F5_{7}
- net MW.K_{0} renamed MW.A0_{0}
- net MW.K_{1} renamed MW.A0_{1}
- net MW.K_{2} renamed MW.A0_{2}
- net MW.K_{3} renamed MW.A0_{3}
- net MW.K_{5} renamed MW.A0_{5}
- net MW.K_{6} renamed MW.A0_{6}
- net MW.K_{7} renamed MW.A0_{7}
- net MW.L_{0} renamed MW.D3_{0}
- net MW.L_{1} renamed MW.D3_{1}
- net MW.L_{2} renamed MW.D3_{2}
- net MW.L_{3} renamed MW.D3_{3}
- net MW.L_{4} renamed MW.D3_{4}
- net MW.L_{5} renamed MW.D3_{5}
- net MW.L_{6} renamed MW.D3_{6}
- net MW.L_{7} renamed MW.D3_{7}
- net MWE_L_{4} renamed MW.H6_{4}
- net MWE_L_{5} renamed MW.H6_{5}
- net MWE_L_{6} renamed MW.H6_{6}
- net MWE_{0} renamed MW.H6_{0}
- net MWE_{1} renamed MW.H6_{1}
- net MWE_{2} renamed MW.H6_{2}
- net MWE_{3} renamed MW.H6_{3}
- net Sys.E58 renamed Sys.E_{58}
- net ~{SEL_E_{0}E_{4}} renamed ~{SEL_H_{L0}H_{L4}}
- net ~{SEL_E_{10}} renamed ~{SEL_H_{L10}}
- net ~{SEL_E_{11}} renamed ~{SEL_H_{L11}}
- net ~{SEL_E_{12}} renamed ~{SEL_H_{L12}}
- net ~{SEL_E_{13}} renamed ~{SEL_H_{L13}}
- net ~{SEL_E_{1}E_{5}} renamed ~{SEL_H_{L1}H_{L5}}
- net ~{SEL_E_{2}E_{6}} renamed ~{SEL_H_{L2}H_{L6}}
- net ~{SEL_E_{3}E_{7}} renamed ~{SEL_H_{L3}H_{L7}}
- net ~{SEL_E_{8}} renamed ~{SEL_H_{L8}}
- net ~{SEL_E_{9}} renamed ~{SEL_H_{L9}}
- new net MW.F5_{1}: U_H13.12, U_J5.16 (Q6), U_K11.3 (A2)
Other:
- note added: "remaining E12 gates appear NC"
- company: (none) -> Meisaka Yukara
- title: (none) -> Centurion VI CPU
- moved on the sheet: R12, R13, U_A15E, U_B12C, U_D10A, U_D10B, U_E12A, U_E12B, U_E12C, U_E12D, U_E12E, U_E12F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
