File: CPU.kicad_sch (KiCad schematic)
At the start: 153 parts, among them P1 Conn_02x36_Top_Bottom, P2 Conn_02x13_Top_Bottom, P3 Conn_02x13_Top_Bottom, P4 Conn_02x08_Counter_Clockwise, P5 Conn_02x25_Counter_Clockwise, P6 Conn_02x25_Counter_Clockwise, P7 Conn_02x07_Counter_Clockwise

Commit message: Revision 12 (see detail), add PDF
* clock control layout changed extensively
* added newly traced pins for address decode
* analysis of address decode
* added newly traced pins for bus control
* layout of bus control updated
* layout of level FF and logic updated
* layout of register index updated
* rename some edge connector pins
* other misc additions from traced pins
Parts:
- R15: value 100k -> 10k
- renumbered RN1 to RN16
Connections:
- net TODO_B12_2 is gone; now on an unnamed net: U_B12.13, U_B12.2, U_C10.11
- net TODO_B15_10_D6_1 is gone; now on net RENAME_B15_D6_M8: U_B15.10 (~{S}), U_D6.1 (S)
- net TODO_B8_3 is gone; now on net PTR.Q_{0}: U_B8.3, U_C7.8
- net TODO_B8_to_B9_B10_19_or_20 is gone; now on net J13_12: U_B8.8
- net TODO_B9_6_Driver is gone; now on net Address.A_{14}: U_A3.11, U_A7.13 (I1b), U_B10.6 (A6), U_B9.6 (A6)
- net TODO_C14_15_GND is gone; now on net GND: U_C14.15 (E)
- net TODO_C14_1_K5 is gone; now on net MW.A0_{7}: U_C14.1 (S)
- net ~{C11_OE2} is gone; now on net ~{Swap_OE}: U_C11.2 (Oe2), U_D4.12 (Q4)
- net +5V: now also U_B10.17 (CS2), U_B15.1 (~{R}), U_B15.13 (~{R}), U_B15.4 (~{S}), U_C15.1 (U/~{D}), U_M9.10 (~{S}), U_M9.12 (D)
- net A13D_a: now also U_A13.13
- net Address.A_{11}: now also U_C8.1
- net Address.A_{12}: now also U_A3.9, U_B10.21 (A4), U_B9.21 (A4)
- net Address.A_{15}: now also U_B10.7 (A7)
- net Address.A_{9}: now also U_C7.5
- net DataF.D_{0}: now also U_C9.3 (D0)
- net DataF.D_{1}: now also U_C9.4 (D1), U_F9.37 (Y1)
- net DataF.D_{2}: now also U_C9.7 (D2)
- net DataF.D_{4}: now also U_C9.13 (D4), U_D9.3 (D0)
- net DataIN.D_{5}: now also U_C12.12 (D2)
- net GND: now also U_B10.19 (~{CS1}), U_C11.15 (Mr), U_C12.15 (Mr), U_C15.10 (~{CET}), U_C15.3 (P0), U_C15.4 (P1), U_C15.5 (P2), U_C15.6 (P3)
- net MW.F5_{4}: now also U_H11.3 (A2)
- net TODO_B8_6: no longer U_B8.6, U_C7.2
- net TODO_E12_4_B10: no longer U_E12.4
- net TODO_M13_12: now also U_A14.13
- net Sys.E_{64}: now reaches P1.64 (Pin_64), RN16.3 (R2), U_A15.13
- net PTR.Q_{7}: now reaches U_A14.4
- net PTR.Q_{7}: now also U_A14.5, U_B10.10 (O0), U_B8.1, U_C8.5
- net at U_C5.15 (~{TC}): now also U_C10.13
- net at JP1.2 (C), JP1.3 (B), U_B12.12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: now also R19.1; no longer R19.2
- net PTR.Q_{6}: now reaches U_A10.14 (IN3), U_B10.12 (O1), U_B11.11, U_B8.4, U_C8.11
- net PTR.Q_{5}: now reaches U_A10.5 (IN1), U_B8.5, U_C7.3
- net PTR.Q_{5}: now also U_B10.14 (O2)
- net at U_C10.10: now also U_A2.12, U_A2.13
- net at U_A8.9 (OE), U_E12.2: no longer R12.1
- net at U_C12.14 (D0), U_D13.5 (O1): now also U_C11.3 (Q0)
- net PTR.Q_{2}: now reaches U_A9.14 (IN3), U_B8.11, U_B9.12 (O1)
- net PTR.Q_{2}: now also U_C7.12
- net PTR.Q_{1}: now reaches U_A9.5 (IN1), U_B9.14 (O2)
- net PTR.Q_{0}: now reaches U_A9.2 (IN0), U_B9.16 (O3)
- net PTR.Q_{0}: now also U_B8.2
- net at U_B10.18 (~{OE}), U_B9.18 (~{OE}): now also U_E12.4
- net CPL_{0}: now reaches U_A8.14 (IN3), U_D9.2 (Q0)
- net CPL_{0}: now also U_C14.13 (I1d)
- net at U_A13.6, U_A13.9: now also U_A13.10
- net CPL_{2}: now reaches U_C14.6 (I1b), U_D10.12, U_D9.15 (Q5)
- net TODO_A1_3_CLOCK: now reaches U_A1.3 (C), U_A3.1
- net ALU.SHIFT_Q0: now reaches U_F9.21 (Q0), U_H6.4 (I2a), U_H6.9 (Zb), U_J10.12 (I7)
- net ALU.CARRY_IN: now reaches U_F6.7 (Za), U_F9.29 (Cn)
- net ALU.SHIFT_RAM0_Q7: now reaches U_F7.16 (Q3), U_F9.9 (RAM0), U_J10.13 (I6)
- net ALU.SHIFT_RAM7: now reaches U_F7.8 (RAM3), U_H6.7 (Za), U_J10.14 (I5)
- net Sys.PA_{17}: now reaches P1.61 (Pin_61), U_A10.15 (BUS3)
- net Sys.PA_{16}: now reaches P1.60 (Pin_60), U_A10.4 (BUS1)
- net ~{Swap_OE}: now reaches U_C11.1 (Oe1), U_C12.1 (Oe1)
- net ~{Swap_OE}: now also U_C12.2 (Oe2)
- net at U_C11.4 (Q1): now also U_C12.13 (D1)
- net at U_B10.13 (D2): now also U_C9.15 (Q5)
- net at U_B10.15 (D3): now also U_C9.12 (Q4)
- net PTR.Q_{4}: now reaches U_B10.16 (O3)
- net PTR.Q_{4}: now also U_B8.6, U_C7.2
- net DataRD_FF: now reaches U_A1.5 (Q), U_A2.1, U_A2.2
- net DataRD_FF: now also U_B12.4
- net A14A_SYS: now reaches U_E15.5 (Q)
- net A14A_SYS: now also U_A14.1, U_A14.2
- net at U_A13.1: now also U_A13.2, U_A13.8
- net ~{DataWR_EN}: now reaches U_A11.9 (BE), U_A12.9 (BE), U_E15.8 (~{Q})
- net Sys.A_is_REGFILE: now reaches P1.47 (Pin_47), U_A2.11
- net B15B_CLK: no longer names the net of U_B15.11 (C), U_E11.6
- net B15_DAT: no longer names the net of U_B11.12, U_B15.12 (D), U_B15.2 (D)
- net ClockB_E8A: no longer names the net of U_E14.13, U_E8.1
- net DataRDCLK renamed DataWRClock
- net DataS.D_{0} renamed MW.E4_{0}
- net DataS.D_{1} renamed MW.E4_{1}
- net DataS.D_{2} renamed MW.E4_{2}
- net DataS.D_{3} renamed MW.E4_{3}
- net DataS.D_{4} renamed MW.E4_{4}
- net DataS.D_{5} renamed MW.E4_{5}
- net DataS.D_{6} renamed MW.E4_{6}
- net DataS.D_{7} renamed MW.E4_{7}
- net M8_I0b renamed RENAME_B15_D6_M8
- net Sys 5MHz renamed Sys.5MHz
- net Sys A_{0} renamed Sys.A_{0}
- net Sys A_{10} renamed Sys.A_{10}
- net Sys A_{12} renamed Sys.PA_{12}
- net Sys A_{13} renamed Sys.PA_{13}
- net Sys A_{14} renamed Sys.PA_{14}
- net Sys A_{15} renamed Sys.CA_{15}
- net Sys A_{1} renamed Sys.A_{1}
- net Sys A_{2} renamed Sys.A_{2}
- net Sys A_{3} renamed Sys.A_{3}
- net Sys A_{4} renamed Sys.A_{4}
- net Sys A_{5} renamed Sys.A_{5}
- net Sys A_{6} renamed Sys.A_{6}
- net Sys A_{7} renamed Sys.A_{7}
- net Sys A_{8} renamed Sys.A_{8}
- net Sys A_{9} renamed Sys.A_{9}
- net Sys D_{0} renamed Sys.D_{0}
- net Sys D_{1} renamed Sys.D_{1}
- net Sys D_{2} renamed Sys.D_{2}
- net Sys D_{3} renamed Sys.D_{3}
- net Sys D_{4} renamed Sys.D_{4}
- net Sys D_{5} renamed Sys.D_{5}
- net Sys D_{6} renamed Sys.D_{6}
- net Sys D_{7} renamed Sys.D_{7}
- net Sys E_{45} renamed Sys.RA_{14}
- net Sys E_{46} renamed Sys.RA_{12}
- net Sys E_{49} renamed Sys.E_{49}
- net Sys E_{50} renamed Sys.E_{50}
- net Sys E_{51} renamed Sys.E_{51}
- net Sys E_{52} renamed Sys.E_{52}
- net Sys RA_{13} renamed Sys.RA_{13}
- net Sys RA_{15} renamed Sys.RA_{15}
- net Sys Reset renamed Sys.Reset
- net Sys.E_{54} renamed Sys.CPL_{0}
- net Sys.E_{55} renamed Sys.CPL_{1}
- net Sys.E_{56} renamed Sys.CPL_{2}
- net Sys.E_{57} renamed Sys.CPL_{3}
- net Sys.E_{58} renamed Sys.RA_{11}
- net TODO_B12_1 renamed J13_12
- net TODO_C14_10 renamed CPL_{1}
- net TODO_C14_3 renamed CPL_{3}
- net VERIFY_A14_6 renamed Sys.~{PTR7_oc}
- net ~{DataREAD_OE} renamed ~{DataRD_EN}
- no-connect marks 39 -> 38
Other:
- note added: "B12A goes LOW when either MMIO or REGFILE are addressed"
- note added: "B12D goes HIGH when REGFILE is addressed OR PTR.Q_{7} is set (high)"
- note added: "B7A output goes LOW when all are true: NOT A_{8} (pending verify) AND NOT A_{9} AND NOT A_{10} AND NOT PA_{11} AND NOT P10_2 (pending verify) AND NOT PA_{13} AND NOT PA_{14} AND NOT PA_{15}(?) AND NOT PA_{16} AND NOT PA_{17} * appears to ignore PA_{12} (unless that's on the P10 connection) * one input is routed to the jumper and R18 * R18 needs to be verified, but is likely pull-UP * this would s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"
- note added: "B8A output goes LOW when all are HIGH: AND PA_{17} AND PA_{16} AND PA_{15}^{(?)} AND PA_{14},PA_{13} AND PA_{11} AND PTR.Q_{7} * ignores PA_{12} * PTR.Q_{7} (high bit) is something I have not studied it has extra functions attached (likely MMIO selection) * this would select (ignoring the high bit): ** 0x3f8nn to 0x3ffnn ** ** 0x3e8nn to 0x3efnn ** * or with the high bit (unlikely as CentVI is a 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"
- note added: "BusCtl Func: DMA?"
- note added: "Counts up from zero (sync-load) Stops at 15"
- note added: "E10C outputs LOW on: Level 1 AND pin9 (TODO)"
- note added: "Edge Top 11 (aka pin47 or Sys.A_is_REGFILE) is OC and follows the output of B7A (pulls LOW when REGFILE addressed)"
- note added: "F14D = (NOT Level=1) AND (SW_H open)"
- note added: "INT ACK ?"
- note added: "PA_{15} ?"
- note added: "Power On Reset"
- note added: "TODO E14_5 to E15?"
- note added: "This could also visually be the trace for pin 5 Which means a different location entirely"
- note added: "this connection is likely wrong"
- note removed: "maybe B12_1 instead"
- moved on the sheet: C39, CR1, JP1, P1, P4, R12, R13, R14, R15, R18, R19, U_A13A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

Commit message: renumbered microcode bits again
Connections:
- net TODO_F7_1: no longer U_F5.12 (Q4), U_F7.1 (A3), U_F9.1 (A3)
- net TODO_F7_2: no longer U_F5.15 (Q5), U_F7.2 (A2), U_F9.2 (A2)
- net TODO_F7_3: no longer U_F5.5 (Q1), U_F7.3 (A1), U_F9.3 (A1)
- net MW.A0_{0} renamed MW.A6_{0}
- net MW.A0_{1} renamed MW.A6_{1}
- net MW.A0_{2} renamed MW.A6_{2}
- net MW.A0_{3} renamed MW.A6_{3}
- net MW.A0_{5} renamed MW.A6_{5}
- net MW.A0_{6} renamed MW.A6_{6}
- net MW.A0_{7} renamed MW.A6_{7}
- net MW.B1_{0} renamed MW.B5_{0}
- net MW.B1_{1} renamed MW.B5_{1}
- net MW.B1_{2} renamed MW.B5_{2}
- net MW.B1_{3} renamed MW.B5_{3}
- net MW.B1_{7} renamed MW.B5_{7}
- net MW.C2_{0} renamed MW.C4_{0}
- net MW.C2_{1} renamed MW.C4_{1}
- net MW.C2_{2} renamed MW.C4_{2}
- net MW.C2_{3} renamed MW.C4_{3}
- net MW.C2_{4} renamed MW.C4_{4}
- net MW.C2_{5} renamed MW.C4_{5}
- net MW.C2_{6} renamed MW.C4_{6}
- net MW.C2_{7} renamed MW.C4_{7}
- net MW.E4_{0} renamed MW.E2_{0}
- net MW.E4_{1} renamed MW.E2_{1}
- net MW.E4_{2} renamed MW.E2_{2}
- net MW.E4_{3} renamed MW.E2_{3}
- net MW.E4_{4} renamed MW.E2_{4}
- net MW.E4_{5} renamed MW.E2_{5}
- net MW.E4_{6} renamed MW.E2_{6}
- net MW.E4_{7} renamed MW.E2_{7}
- net MW.F5_{0} renamed MW.F1_{0}
- net MW.F5_{1} renamed MW.F1_{1}
- net MW.F5_{2} renamed MW.F1_{2}
- net MW.F5_{3} renamed MW.F1_{3}
- net MW.F5_{4} renamed MW.F1_{4}
- net MW.F5_{5} renamed MW.F1_{5}
- net MW.F5_{6} renamed MW.F1_{6}
- net MW.F5_{7} renamed MW.F1_{7}
- net MW.H6_{0} renamed MW.H0_{0}
- net MW.H6_{1} renamed MW.H0_{1}
- net MW.H6_{2} renamed MW.H0_{2}
- net MW.H6_{3} renamed MW.H0_{3}
- net MW.H6_{4} renamed MW.H0_{4}
- net MW.H6_{5} renamed MW.H0_{5}
- net MW.H6_{6} renamed MW.H0_{6}
- net MW.H6_{7} renamed MW.H0_{7}
- new net MW.B5_{4}: U_F5.12 (Q4)
- new net MW.B5_{5}: U_F5.15 (Q5)
- new net MW.B5_{6}: U_F5.5 (Q1)

Commit message: rename a bunch of signals
Connections:
- net at U_M14.2 (I0a), U_M15.2 (I0a): now also U_M12.2 (Q0)
- net A10_OE renamed AddrHToSys
- net B12_~{F13_D_{0}} renamed INT_ENABLE
- net DataIN.D_{0} renamed DataP.D_{0}
- net DataIN.D_{1} renamed DataP.D_{1}
- net DataIN.D_{2} renamed DataP.D_{2}
- net DataIN.D_{3} renamed DataP.D_{3}
- net DataIN.D_{4} renamed DataP.D_{4}
- net DataIN.D_{5} renamed DataP.D_{5}
- net DataIN.D_{6} renamed DataP.D_{6}
- net DataIN.D_{7} renamed DataP.D_{7}
- net F14C_a renamed RTC_INT
- net F14C_b renamed RTC_INT_EN
- net ~{A4_INE} renamed ~{AddrLToData}
- net ~{A7_EN_B} renamed ~{AddrMToData}
- net ~{A7_OEa_M7_OEa} renamed ~{DSWh_INT_OE}
- net ~{C13_EN} renamed ~{RIndex_LD}
- net ~{C9_EN} renamed ~{Result_LD}
- net ~{D11_EN} renamed ~{PTIndex_LD}
- net ~{D13_OE} renamed ~{Reg_OE}
- net ~{D9_EN} renamed ~{Level_LD}
- net ~{M6_OE} renamed ~{MWConst_OE}
- net ~{M7_OEb} renamed ~{SenseSW_OE}
- net ~{SenseSW_OE}: no longer U_M12.2 (Q0)
Other:
- note added: "DataP ?"

Commit message: naming and bus fixups
Parts:
- removed R4: 330, Resistor_THT:R_Array_SIP10, symbol Device:R_Network09
- removed RN16: R_Network09, Resistor_THT:R_Array_SIP10, symbol Device:R_Network09
- added R4, RN16: 220/330, Resistor_THT:R_Array_SIP10, symbol Device:R_Network_Dividers_x08_SIP
- XTAL1: value 5.000MHz -> 15.000MHz
Connections:
- net DataB.D_{0} is gone; now on net DataF.D_{0}: U_A11.17 (A3), U_B13.6 (Q0), U_C13.3 (D0)
- net DataB.D_{1} is gone; now on net DataF.D_{1}: U_A11.13 (A2), U_B13.7 (Q1), U_C13.8 (D3), U_D11.4 (D1)
- net DataB.D_{4} is gone; now on net DataF.D_{4}: U_A12.17 (A3), U_B13.11 (Q4), U_C13.13 (D4)
- net Sys.E_{49} is gone; now on net Sys.INR0: P1.49 (Pin_49)
- net +5V: now also R4.10 (COM2), RN16.10 (COM2)
- net DataF.D_{2}: now also U_B13.8 (Q2), U_C13.7 (D2)
- net DataF.D_{3}: now also U_B13.9 (Q3), U_C13.4 (D1)
- net DataF.D_{5}: now also U_B13.12 (Q5), U_C13.14 (D5)
- net DataF.D_{6}: now also U_B13.13 (Q6), U_C13.17 (D6)
- net DataF.D_{7}: now also U_B13.14 (Q7), U_C13.18 (D7); no longer U_C13.19 (Q7), U_C14.2 (I0a)
- net F13_D_{1}: now also R4.6 (R5)
- net FPC_P2_12: now also R4.5 (R4)
- net GND: now also R4.1 (COM1), RN16.1 (COM1)
- net R4_7: now also R4.7 (R6)
- net SW_2: now also R4.8 (R7)
- net Sys.E_{63}: now also RN16.5 (R4)
- net Sys.E_{64}: now also RN16.3 (R2)
- net at U_A14.3: now also RN16.2 (R1)
- net Sys.~{DRDY}: now reaches P1.44 (Pin_44), U_A2.8, U_A3.3
- net at P2.11 (Pin_11), U_M8.6 (I2a): now also R4.2 (R1)
- net at P2.10 (Pin_10), U_M8.8 (I3a): now also R4.3 (R2)
- net at P3.13 (Pin_13), U_M9.11 (C): now also R4.4 (R3)
- net Sys.~{RDIN}: now reaches P1.42 (Pin_42), U_A2.3
- net Sys.~{WTIN}: now reaches P1.43 (Pin_43), U_A2.6
- net ~{ALU_Flags_EN}: now reaches U_E7.13 (O2)
- net ~{ALU_Flags_EN}: now also U_J9.1 (~{E})
- net A1_6-B11_3 renamed ~{DataRDCycle}
- net A1_8-B11_4 renamed ~{DataWTCycle}
- net A7_6 renamed Sys.INR0
- net Sys.INR0: now also RN16.7 (R6)
- net CLOCK_COUNT_15 renamed BUS_TIMEOUT
- net DataRD_FF renamed DataRDCycle
- net DataWRClock renamed DataWTClock
- net H12_~{S} renamed ~{DataReady}
- net Sys.A_is_REGFILE renamed Sys.~{APRE}
- net Sys.E_{50} renamed Sys.INR1
- net Sys.INR1: now also RN16.8 (R7)
- net Sys.E_{51} renamed Sys.INR2
- net Sys.INR2: now also RN16.9 (R8)
- net Sys.E_{52} renamed Sys.INR3
- net Sys.INR3: now also RN16.6 (R5)
- net Sys.RA_{11} renamed Sys.~{RA_{11}}
- net Sys.RA_{12} renamed Sys.~{RA_{12}}
- net Sys.RA_{13} renamed Sys.~{RA_{13}}
- net Sys.RA_{14} renamed Sys.~{RA_{14}}
- net Sys.RA_{15} renamed Sys.~{RA_{15}}
- net ~{B13_EN} renamed ~{MAPROM_SEL}
- net ~{DataWR_EN} renamed ~{DataWT_EN}
- new net: U_C13.19 (Q7), U_C14.2 (I0a)
Other:
- note added: "Carry Bit Select"
- note added: "Clock Control and Gating"
- note added: "Datapath Select"
- note added: "Edge Top 11 (aka pin47 or Sys.~{APRE}) is OC and follows the output of B7A (pulls LOW when REGFILE addressed)"
- note added: "Interrupt Control"
- note added: "Level"
- note added: "Microcode Constant/Gate"
- note added: "Nibble Swap"
- note added: "Page Bank"
- note added: "Register Data Latch"
- note added: "Result Select"
- note added: "Shift Bit Select"
- note added: "System Databus"
- note added: "Write Control"
- note added: "these three pins drive the register file index their order does not matter after this point"
- note removed: "Edge Top 11 (aka pin47 or Sys.A_is_REGFILE) is OC and follows the output of B7A (pulls LOW when REGFILE addressed)"
- note removed: "this connection is likely wrong"
- moved on the sheet: R7, U_A2B

Commit message: some much needed improvements to bus connections
Connections:
- net AddrB.A_{8} is gone; now on net M15_I1b: U_B10.4 (A0), U_B9.4 (A0), U_D11.7 (Q2)
- net D13_12_F9_25 is gone; now on net DataP.D_{0}: U_D13.12 (O4), U_F9.25 (D0), U_H14.9 (O4a)
- net D13_9_F7_25 is gone; now on net DataP.D_{4}: U_D13.9 (O3), U_F7.25 (D0)
- net DataA_{0} is gone; now on net Res.D_{0}: U_B3.13 (I1d)
- net DataA_{1} is gone; now on net Res.D_{1}: U_B3.10 (I1c)
- net DataA_{3} is gone; now on net Res.D_{3}: U_B3.3 (I1a), U_B4.3 (I1a)
- net +5V: now also U_J10.1 (I3), U_J11.3 (I1)
- net DataP.D_{0}: now also U_M6.3 (O3b), U_M7.12 (O3a), U_M7.9 (O0b)
- net DataP.D_{1}: now also U_M6.5 (O2b), U_M7.14 (O2a), U_M7.7 (O1b)
- net DataP.D_{2}: now also U_F9.23 (D2), U_H14.5 (O2a), U_M6.7 (O1b), U_M7.16 (O1a), U_M7.5 (O2b)
- net DataP.D_{3}: now also U_M6.9 (O0b), U_M7.18 (O0a), U_M7.3 (O3b)
- net DataP.D_{4}: now also U_M14.12 (O3a), U_M6.18 (O0a)
- net DataP.D_{5}: now also U_M14.14 (O2a), U_M6.16 (O1a)
- net DataP.D_{6}: now also U_C11.3 (Q0), U_C12.14 (D0), U_D13.5 (O1), U_M14.16 (O1a), U_M6.14 (O2a)
- net DataP.D_{7}: now also U_M14.18 (O0a), U_M6.12 (O3a)
- net Sys.INR3: no longer U_A7.18 (O0a), U_A8.3 (OUT0)
- net TODO_K13_10_F9_31: now reaches U_K13.10 (I0b)
- net TODO_K13_10_F9_31: now also U_F9.31 (F3)
- net TODO_K13_11_F13_12: now reaches U_K13.11 (I1b)
- net TODO_K13_11_F13_12: now also U_F13.12 (Q4), U_H13.5
- net TODO_K13_13_B15: now reaches U_K13.13 (I3b)
- net TODO_J12_10_M12_2: now reaches U_M12.2 (Q0), U_M14.2 (I0a), U_M15.2 (I0a)
- net TODO_J12_10_M12_2: now also U_J12.10 (I0b)
- net TODO_J12_6_M12_5: now reaches U_M14.4 (I1a), U_M15.4 (I1a)
- net TODO_J12_6_M12_5: now also U_J12.6 (I0a), U_M12.5 (Q1); no longer U_M12.4 (D1)
- net CCR.OVER: now reaches P3.2 (Pin_2), U_J11.13 (I6), U_J11.2 (I2), U_M12.7 (Q2), U_M14.6 (I2a), U_M15.6 (I2a)
- net Res.D_{1}: now reaches U_B4.10 (I1c)
- net Res.D_{1}: now also U_B9.13 (D2), U_C9.5 (Q1)
- net Res.D_{0}: now reaches U_B4.13 (I1d)
- net Res.D_{0}: now also U_B9.15 (D3), U_C9.2 (Q0), U_D15.15 (D3)
- net Res.D_{3}: now reaches U_B9.9 (D0), U_C9.9 (Q3)
- net TODO_J12_11_J9_2: now reaches U_J12.11 (I1b), U_J13.10 (I0b)
- net TODO_J12_11_J9_2: now also U_J9.14 (D5), U_J9.2 (Q0), U_K10.1
- net Res.D_{5}: now reaches U_C4.10 (I1c)
- net Res.D_{5}: now also U_B10.13 (D2), U_C3.10 (I1c), U_C9.15 (Q5), U_D14.13 (D2)
- net Res.D_{4}: now reaches U_C4.13 (I1d)
- net Res.D_{4}: now also U_B10.15 (D3), U_C3.13 (I1d), U_C9.12 (Q4), U_D14.15 (D3), U_J10.15 (I4)
- net Res.D_{7}: now reaches U_C3.3 (I1a), U_C4.3 (I1a)
- net Res.D_{7}: now also U_B10.9 (D0), U_C9.19 (Q7), U_D14.9 (D0), U_J12.12 (I2b)
- net Res.D_{6}: now reaches U_B10.11 (D1), U_C3.6 (I1b), U_C4.6 (I1b), U_C9.16 (Q6)
- net Res.D_{6}: now also U_D14.11 (D1), U_J12.4 (I2a)
- net TODO_M12_4_J12_7: now reaches U_J12.7 (Za)
- net TODO_M12_4_J12_7: now also U_M12.4 (D1)
- net DataA_{2} renamed Res.D_{2}
- net SEQ.~{ZERO} renamed ~{Reset_{1}}
- new net: U_A7.18 (O0a), U_A8.3 (OUT0)
Other:
- note added: "Constants are inverted!"
- note added: "E8.12 ?"
- note added: "F"
- note added: "Frontpanel Driver"
- note added: "L"
- note added: "M"
- note added: "V"
- note removed: "DataP ?"
- note removed: "Frontpanel Drivers"

Commit message: a substantial layout refactor
also a subtle visual convention which almost no one will notice
Connections:
- net ALU.CARRY is gone; now on net TODO_J9_11_F7_33: U_F7.33 (Cn+4), U_H6.3 (I3a)
- net ALU.ZERO is gone; now on net TODO_F7_11_F9_11: R5.2, U_F9.11 (F=0), U_J9.3 (D0)
- net PTR.Q_{1} is gone; now on net P10_2: U_A9.5 (IN1), U_B9.14 (O2)
- net PTR.Q_{4} is gone; now on net TODO_A10_2_B10_16: U_B10.16 (O3), U_B8.6, U_C7.2
- net PTR.Q_{7} is gone; now on net P10_8: U_A14.4, U_A14.5, U_B10.10 (O0), U_B8.1, U_C8.5
- net +5V: now also U_D7.16 (Vcc), U_M12.16 (VCC), U_M13.16 (VCC), U_M14.20 (VCC), U_M15.20 (VCC); no longer U_H12.12 (~{R}), U_H12.4 (~{R}), U_J10.1 (I3), U_J11.3 (I1)
- net Address.A_{12}: now also U_A7.17 (I3b)
- net Address.A_{15}: now also U_A7.11 (I0b)
- net Address.A_{9}: now also U_A6.5 (IN1)
- net CCR.OVER: no longer P3.2 (Pin_2)
- net DataF.D_{0}: now also U_D11.6 (D2)
- net DataF.D_{2}: now also U_D11.3 (D0)
- net DataP.D_{1}: now also U_F9.24 (D1)
- net DataP.D_{2}: now also U_A6.10 (OUT2), U_A9.13 (OUT3)
- net DataP.D_{3}: now also U_A6.13 (OUT3), U_F9.22 (D3)
- net DataP.D_{5}: now also U_A5.6 (OUT1), U_A7.14 (O2a), U_A7.5 (O2b), U_A8.10 (OUT2), U_F7.24 (D1)
- net DataP.D_{6}: now also U_A5.13 (OUT3), U_A7.16 (O1a), U_A7.7 (O1b), U_A8.6 (OUT1), U_F7.23 (D2)
- net DataP.D_{7}: now also U_A10.10 (OUT2), U_A12.2 (R0), U_A5.10 (OUT2), U_A7.18 (O0a), U_A7.9 (O0b), U_A8.3 (OUT0), U_F7.22 (D3)
- net MW.A6_{0}: now also U_F7.3 (A1), U_F9.3 (A1)
- net MW.A6_{1}: now also U_F7.2 (A2), U_F9.2 (A2)
- net MW.A6_{2}: now also U_F7.1 (A3), U_F9.1 (A3)
- net MW.B5_{2}: now also U_F9.6 (I_8)
- net MW.B5_{3}: now also U_F11.13 (D), U_F7.17 (B0), U_F9.17 (B0), U_M13.13 (D)
- net MW.B5_{4}: now also U_F11.1 (A0), U_F7.18 (B1), U_F9.18 (B1), U_M13.1 (A0)
- net MW.B5_{5}: now also U_F11.2 (A1), U_F7.19 (B2), U_F9.19 (B2), U_M13.2 (A1)
- net MW.B5_{6}: now also U_F11.3 (A2), U_F7.20 (B3), U_F9.20 (B3), U_M13.3 (A2)
- net MW.C4_{2}: now also U_F9.12 (I_0)
- net MW.C4_{4}: now also U_F9.14 (I_2)
- net MW.C4_{5}: now also U_F7.26 (I_3), U_F9.26 (I_3)
- net MW.C4_{6}: now also U_F7.28 (I_4), U_F9.28 (I_4)
- net MW.C4_{7}: now also U_F9.27 (I_5)
- net FP.~{ABT}: now reaches P3.16 (Pin_16), R1.1
- net FP.~{RUN}: now reaches U_M14.17 (I3b), U_M14.5 (O2b)
- net FP.~{RUN}: now also P3.2 (Pin_2)
- net FP.~{HALT}: now reaches P3.1 (Pin_1), U_M14.3 (O3b)
- net FP.RTI: now reaches P3.13 (Pin_13), R4.4 (R3), U_M9.11 (C)
- net AFL.HALFC: now reaches U_J13.5 (I1a), U_J9.12 (Q4)
- net AFL.LZERO: now reaches U_J9.15 (Q5), U_K10.2
- net TODO_F7_11_F9_11: now reaches U_F7.11 (F=0)
- net Sys.PA_{15}: now reaches P1.59 (Pin_59), U_A10.1 (BUS0)
- net TODO_A10_2_B10_16: now reaches U_A10.2 (IN0)
- net AFL.OVER: now reaches U_J11.9 (S2), U_J9.7 (Q2)
- net ~{M13_EN}: now reaches U_M13.14 (E)
- net ~{M13_EN}: now also U_K11.13 (O2)
- net AFL.SIGN: now reaches U_J12.3 (I3a), U_J12.5 (I1a), U_J9.5 (Q1)
- net TODO_J9_11_F7_33: now reaches U_J9.11 (D3)
- net ClockA: no longer names the net of U_E10.2, U_E11.3, U_H12.6 (Y)
- net ClockB: no longer names the net of U_E10.13, U_E8.5, U_E8.6, U_H12.10 (Y), U_J6.1, U_K10.4, U_K10.5
- net F11_EN renamed ~{F11_EN}
- net M15_I1b renamed Page.B_{0}
- net M15_I2b renamed Page.B_{1}
- net M15_I3b renamed Page.B_{2}
- net M8_I3b renamed RENAME_MODECTL
- net MainClockPhi2 renamed ~{MainClockPhi1}
- net SEQ.MC_CLK renamed ~{ClockB_{0}}
- net ~{A1_E15_F12_RESET} renamed ~{Reset_{2}}
- new net TODO_H12_4,12: U_H12.12 (~{R}), U_H12.4 (~{R})
- new net TODO_VCC: U_J10.1 (I3), U_J11.3 (I1)
Other:
- note added: "ALU Flags"
- note added: "B7A output goes LOW when all are true: NOT A_{8} (pending verify) AND NOT A_{9} AND NOT A_{10} AND NOT PA_{11} AND NOT P10_2 (pending verify as PA_{12}) AND NOT PA_{13} AND NOT PA_{14} AND NOT PA_{15}(?) AND NOT PA_{16} AND NOT PA_{17} * PA_{12} is probably on the U_C7C.9 (P10_2) connection * one input is routed to the jumper and R18 * R18 needs to be verified, but is likely pull-UP * this would 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"
- note added: "B8A output goes LOW when all are HIGH: AND PA_{17} AND PA_{16} AND PA_{15}^{(?)} AND PA_{14},PA_{13} AND PA_{11} AND PTR.Q_{7} * ignores PA_{12} * PTR.Q_{7} (high bit) has extra memory functions attached (likely page control and MMIO selection) * this would select (ignoring the high bit): ** 0x3f8nn to 0x3ffnn ** ** 0x3e8nn to 0x3efnn **"
- note added: "Carry Select"
- note added: "F14D = LOW IF (Level=1 OR SW_H=closed)"
- note added: "Fault Select"
- note added: "ISA Index ROM"
- note added: "Link Select"
- note added: "Microcode JSR Select"
- note added: "Register Data"
- note added: "Register Index"
- note added: "Result Register"
- note added: "Shift Select"
- note added: "System Data Bus"
- note added: "ZERO is an OC line"
- note added: "does M8.12 float? or is the cross connect wrong?"
- note added: "maybe F12"
- note added: "maybe F12 -> H14"
- note added: "probably GND?"
- note removed: "ALU Result"
- note removed: "B7A output goes LOW when all are true: NOT A_{8} (pending verify) AND NOT A_{9} AND NOT A_{10} AND NOT PA_{11} AND NOT P10_2 (pending verify) AND NOT PA_{13} AND NOT PA_{14} AND NOT PA_{15}(?) AND NOT PA_{16} AND NOT PA_{17} * appears to ignore PA_{12} (unless that's on the P10 connection) * one input is routed to the jumper and R18 * R18 needs to be verified, but is likely pull-UP * this would s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"
- note removed: "B8A output goes LOW when all are HIGH: AND PA_{17} AND PA_{16} AND PA_{15}^{(?)} AND PA_{14},PA_{13} AND PA_{11} AND PTR.Q_{7} * ignores PA_{12} * PTR.Q_{7} (high bit) is something I have not studied it has extra functions attached (likely MMIO selection) * this would select (ignoring the high bit): ** 0x3f8nn to 0x3ffnn ** ** 0x3e8nn to 0x3efnn ** * or with the high bit (unlikely as CentVI is a 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"
- note removed: "Carry Bit Select"
- note removed: "F14D = (NOT Level=1) AND (SW_H open)"
- note removed: "Register Data Latch"
- note removed: "Result Store"
- note removed: "Shift Bit Select"
- note removed: "System Databus"
- note removed: "These may be the Address bus but traces for them are not visible"
- moved on the sheet: BODGE1, P4, R12, R14, R17, R2, R3, R5, R6, R8, R9, U_A15E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
