File: CPU.kicad_sch (KiCad schematic)
At the start: 153 parts, among them P1 Conn_02x36_Top_Bottom, P2 Conn_02x13_Top_Bottom, P3 Conn_02x13_Top_Bottom, P4 Conn_02x08_Counter_Clockwise, P5 Conn_02x25_Counter_Clockwise, P6 Conn_02x25_Counter_Clockwise, P7 Conn_02x07_Counter_Clockwise

Commit message: more pins! more progress!
Connections:
- net K9_In3 is gone; now on net REG_MMIO: U_B12.3, U_K9.1 (I3)
- net TODO_A10_2_B10_16 is gone; now on net PTR.Q_{4}: U_A10.2 (IN0), U_B10.16 (O3), U_B8.6, U_C7.2
- net TODO_B7_5 is gone; now on an unnamed net: U_B7.5, U_B7.6
- net TODO_D12_2_D8_8 is gone; now on net DMAWrite: U_D12.2, U_D8.9
- net TODO_D7_11_M6_16 is gone; now on net ~{MainClockPhi1}: U_D7.11 (CP), U_D7.5 (CP)
- net TODO_D8_1 is gone; now on net DMARead: U_D12.13, U_D8.1
- net TODO_E10_12_E14_3 is gone; now on net ~{DataEndCycle}: U_E10.12, U_E14.3, U_E15.3 (C)
- net TODO_E14_9 is gone; now on net SysDataRD: U_E11.11, U_E14.9
- net TODO_F14_F13 is gone; now on an unnamed net: U_F14.4, U_F14.5
- net TODO_H12_4,12 is gone; now on net GND: U_H12.12 (~{R}), U_H12.4 (~{R})
- net TODO_J10_2_H6_11 is gone; now on net AFL.CARRY: U_H6.11 (I1b), U_H6.5 (I1a), U_J10.2 (I2), U_J9.10 (Q3)
- net TODO_K13_13_B15 is gone; now on net GND: U_K13.13 (I3b)
- net TODO_K9_2or15or14_D10_6 is gone; now on an unnamed net: U_D10.6
- net WorkAddr_Clock is gone; now on net C15_~{PE}: U_D6.10 (I1c)
- net ~{FPC_P2_M8_12} is gone; now on net DMAStartCycle: U_D8.10, U_D8.5, U_M8.12 (O3a)
- net +5V: now also R14.2, U_D14.17 (CS2), U_D15.17 (CS2), U_F12.10 (~{S}), U_F12.13 (~{R}), U_F13.1 (~{Mr}), U_F6.5 (I1a), U_H6.13 (I3b), U_J11.12 (I7), U_J11.14 (I5), U_J11.3 (I1)
- net AFL.OVER: now also U_J13.11 (I1b)
- net AFL.SIGN: now also U_J13.6 (I0a)
- net CPL_{1}: now also U_A8.11 (IN2)
- net CPL_{2}: now also U_A8.5 (IN1)
- net CPL_{3}: now also U_A8.2 (IN0)
- net DataF.D_{2}: now also U_A11.7 (A1)
- net DataF.D_{3}: now also U_A11.3 (A0)
- net DataF.D_{5}: now also U_A12.13 (A2)
- net DataF.D_{6}: now also U_A12.7 (A1)
- net DataF.D_{7}: now also U_A12.3 (A0)
- net DataP.D_{0}: now also U_A4.3 (OUT0)
- net DataP.D_{1}: now also U_A4.6 (OUT1), U_C11.12 (D2), U_C12.5 (Q2), U_D13.15 (O5), U_H14.7 (O3a)
- net DataP.D_{2}: now also U_A4.13 (OUT3), U_D13.16 (O6)
- net DataP.D_{3}: now also U_A4.10 (OUT2), U_D13.19 (O7), U_H14.3 (O1a)
- net DataP.D_{5}: now also U_D13.6 (O2)
- net DataP.D_{7}: now also U_D13.2 (O0)
- net E10_8_F14_2: now also U_H14.2 (I1)
- net GND: now also U_D14.18 (~{OE}), U_D14.19 (~{CS1}), U_D15.18 (~{OE}), U_D15.19 (~{CS1}), U_D7.12 (~{R}), U_D7.4 (~{R}), U_E15.12 (D), U_E15.2 (D), U_F12.2 (D), U_F6.1 (Ea), U_F6.3 (I3a), U_F6.6 (I0a), U_H12.15 (M), U_H14.4 (I2), U_H6.10 (I0b), U_J11.1 (I3), U_J13.13 (I3b), U_J13.3 (I3a), U_K13.3 (I3a), U_L9.4 (D_{3})
- net INT_ENABLE: now also U_C10.5, U_K13.10 (I0b)
- net MW.D3_{0}: now also U_J10.9 (S2), U_L9.7 (D_{0})
- net MW.D3_{1}: now also U_L9.6 (D_{1})
- net MW.D3_{2}: now also U_L9.5 (D_{2})
- net P10_8: now also U_H14.10 (I4); no longer U_D12.1, U_K9.15 (I4)
- net P4_7: now also R12.2
- net PTR.Q_{5}: now also U_B11.10
- net Res.D_{1}: now also U_D15.13 (D2)
- net Res.D_{2}: now also U_D15.11 (D1)
- net Res.D_{3}: now also U_D15.9 (D0)
- net Res.D_{5}: now also U_J11.15 (I4), U_J11.4 (I0)
- net Sys.~{DRDY}: now also RN16.2 (R1), U_A14.3
- net TODO_M12_11_J10: now also U_J10.5 (Z)
- net TODO_VCC: no longer U_J11.3 (I1)
- net ~{AddrLToData}: now also U_A5.7 (INE)
- net at U_E10.5: now also U_B15.9 (Q)
- net MWS.A_{7}: now reaches U_MWE2.1 (A7), U_MWF2.1 (A7), U_MWH2.1 (A7), U_MWJ2.1 (A7), U_MWK2.1 (A7), U_MWL2.1 (A7), U_MWM2.1 (A7)
- net MWS.A_{7}: now also U_J7.21 (Y_{3})
- net MWS.A_{6}: now reaches U_MWE2.2 (A6), U_MWF2.2 (A6), U_MWH2.2 (A6), U_MWJ2.2 (A6), U_MWK2.2 (A6), U_MWL2.2 (A6), U_MWM2.2 (A6)
- net MWS.A_{6}: now also U_J7.20 (Y_{2})
- net MWS.A_{10}: now reaches U_MWE2.21 (A10), U_MWF2.21 (A10), U_MWH2.21 (A10), U_MWJ2.21 (A10), U_MWK2.21 (A10), U_MWL2.21 (A10), U_MWM2.21 (A10)
- net MWS.A_{10}: now also U_L9.14 (Y_{2})
- net MWS.A_{9}: now reaches U_MWE2.22 (A9), U_MWF2.22 (A9), U_MWH2.22 (A9), U_MWJ2.22 (A9), U_MWK2.22 (A9), U_MWL2.22 (A9), U_MWM2.22 (A9)
- net MWS.A_{9}: now also U_L9.13 (Y_{1})
- net MWS.A_{8}: now reaches U_MWE2.23 (A8), U_MWF2.23 (A8), U_MWH2.23 (A8), U_MWJ2.23 (A8), U_MWK2.23 (A8), U_MWL2.23 (A8), U_MWM2.23 (A8)
- net MWS.A_{8}: now also U_L9.12 (Y_{0})
- net MWS.A_{5}: now reaches U_MWE2.3 (A5), U_MWF2.3 (A5), U_MWH2.3 (A5), U_MWJ2.3 (A5), U_MWK2.3 (A5), U_MWL2.3 (A5), U_MWM2.3 (A5)
- net MWS.A_{5}: now also U_J7.19 (Y_{1})
- net MWS.A_{4}: now reaches U_MWE2.4 (A4), U_MWF2.4 (A4), U_MWH2.4 (A4), U_MWJ2.4 (A4), U_MWK2.4 (A4), U_MWL2.4 (A4), U_MWM2.4 (A4)
- net MWS.A_{4}: now also U_J7.18 (Y_{0})
- net MWS.A_{3}: now reaches U_MWE2.5 (A3), U_MWF2.5 (A3), U_MWH2.5 (A3), U_MWJ2.5 (A3), U_MWK2.5 (A3), U_MWL2.5 (A3), U_MWM2.5 (A3)
- net MWS.A_{3}: now also U_K7.21 (Y_{3})
- net MWS.A_{2}: now reaches U_MWE2.6 (A2), U_MWF2.6 (A2), U_MWH2.6 (A2), U_MWJ2.6 (A2), U_MWK2.6 (A2), U_MWL2.6 (A2), U_MWM2.6 (A2)
- net MWS.A_{2}: now also U_K7.20 (Y_{2})
- net MWS.A_{1}: now reaches U_MWE2.7 (A1), U_MWF2.7 (A1), U_MWH2.7 (A1), U_MWJ2.7 (A1), U_MWK2.7 (A1), U_MWL2.7 (A1), U_MWM2.7 (A1)
- net MWS.A_{1}: now also U_K7.19 (Y_{1})
- net MWS.A_{0}: now reaches U_MWE2.8 (A0), U_MWF2.8 (A0), U_MWH2.8 (A0), U_MWJ2.8 (A0), U_MWK2.8 (A0), U_MWL2.8 (A0), U_MWM2.8 (A0)
- net MWS.A_{0}: now also U_K7.18 (Y_{0})
- net at U_E14.12: now also U_E15.4 (~{S})
- net PTR.~{Q_{7}}: now reaches JP1.2 (C), JP1.3 (B), R19.1, U_B12.12, U_C8.6
- net PTR.~{Q_{7}}: now also U_D12.4, U_D8.13, U_J13.4 (I2a)
- net at U_E11.2, U_E14.2: now also U_E11.1
- net WorkAddr_TC: now reaches U_C10.12
- net WorkAddr_TC: now also U_D12.9
- net DMA_P2_12: now reaches U_M14.9 (O0b)
- net DMA_P2_12: now also U_E10.9
- net at U_D13.13 (D4): now also U_D15.16 (O3)
- net DMAWrite: now reaches P2.11 (Pin_11), R4.2 (R1), U_M8.6 (I2a)
- net DMAStartCycle: now reaches U_D8.4
- net FPC_P3_9: now reaches P3.9 (Pin_9)
- net FPC_P3_9: now also U_H14.6 (I3)
- net PTR.Q_{4}: now reaches U_B11.9
- net at U_E14.5: now also U_E14.4
- net REG_MMIO: now reaches U_D12.12
- net K9_In4: now reaches U_B12.11
- net K9_In4: now also U_D12.1, U_K9.15 (I4)
- net SysDataRD: now reaches U_E7.12 (O3), U_E8.12
- net DMARead: now reaches U_M8.14 (O2a)
- net DMARead: now also U_E11.4
- net AFL.CARRY: now reaches U_F6.4 (I2a)
- net A14A_SYS renamed BUS_FORCE_READY
- net F12B_D: no longer names the net of U_C10.4, U_D6.3 (I1a), U_F12.12 (D)
- net F13_D_{1} renamed ~{DMA_P2_13}
- net FPC_P2_12 renamed ~{DMA_P2_12}
- removed net J11_IN_{0}_IN_{4}: U_F12.6 (~{Q}), U_J11.15 (I4), U_J11.4 (I0)
- net K9_In0 renamed CondCycle
- net K9_In1 renamed CondRIR_{0NOR4}
- net RENAME_B15_D6_M8 renamed DMAAddressControl
- net Sys.CPL_{0} renamed Sys.~{CPL_{0}}
- net Sys.CPL_{1} renamed Sys.~{CPL_{1}}
- net Sys.CPL_{2} renamed Sys.~{CPL_{2}}
- net Sys.CPL_{3} renamed Sys.~{CPL_{3}}
- net TODO_A1_3_CLOCK renamed ~{DataEndCycle}
- net TODO_A5_5 renamed Address.A_{5}
- net TODO_E10_9 renamed CCR.CARRY
- net CCR.CARRY: no longer U_E10.9
- net TODO_J12_6_M12_5 renamed TODO_M12_5_M14
- net TODO_J9_11_F7_33 renamed ALU.CARRY
- net TODO_K13_10_F9_31: no longer names the net of U_F9.31 (F3)
- net TODO_K13_10_F9_31: no longer U_K13.10 (I0b)
- net TODO_K9_D10_5 renamed CondRIR_{0}
- net ~{A1A_S}: no longer names the net of U_A1.4 (~{S}), U_D7.9 (~{Y})
- net ~{A1B_SET}: no longer names the net of U_A1.10 (~{S}), U_D7.7 (~{Y}), U_F12.4 (~{S})
- no-connect marks 38 -> 52
Other:
- note added: "B12A goes HIGH when either MMIO or REGFILE are addressed"
- note added: "B12D is HIGH when REGFILE is addressed OR PTR.Q_{7} is set (high) LOW when Memory is addressed AND PTR.Q_{7} is clear (low)"
- note added: "B7A output goes LOW when all are true: NOT A_{8} AND NOT A_{9} AND NOT A_{10} AND NOT PA_{11} AND NOT PA_{12} AND NOT PA_{13} AND NOT PA_{14} AND NOT PA_{15} AND NOT PA_{16} AND NOT PA_{17} * one input is routed to the jumper and R18 * R18 needs to be verified, but is likely pull-UP * this would select addresses in: ** 0x000rr ** * if JP1 has 1+2 jumped, an extra signal: PTR.Q_{7} is included thi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"
- note added: "E10C outputs LOW on: (Level is 0 or 1) AND INT_ENABLE AND P2.12 pulled LOW"
- note added: "F14D = LOW IF (SW_H=open AND DMA_INT_Request?) typically HIGH"
- note added: "Microcode Sequence Low -> Hi"
- note added: "checking pin 15 could finalize NC half"
- note added: "it's unclear which side of JP1 is connected to this net"
- note added: "needs re-verify pin5/6 is very important here if pin 5, then 1 is VCC if pin 6, then 1 is GND this is needed for SF/RF to work"
- note removed: "B12A goes LOW when either MMIO or REGFILE are addressed"
- note removed: "B12D goes HIGH when REGFILE is addressed OR PTR.Q_{7} is set (high)"
- note removed: "B7A output goes LOW when all are true: NOT A_{8} (pending verify) AND NOT A_{9} AND NOT A_{10} AND NOT PA_{11} AND NOT P10_2 (pending verify as PA_{12}) AND NOT PA_{13} AND NOT PA_{14} AND NOT PA_{15}(?) AND NOT PA_{16} AND NOT PA_{17} * PA_{12} is probably on the U_C7C.9 (P10_2) connection * one input is routed to the jumper and R18 * R18 needs to be verified, but is likely pull-UP * this would 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"
- note removed: "E10C outputs LOW on: Level 1 AND pin9 (TODO)"
- note removed: "E8.12 ?"
- note removed: "F14D = LOW IF (Level=1 OR SW_H=closed)"
- note removed: "Microcode Sequence Low > Hi"
- note removed: "PA_{15} ?"
- note removed: "TODO E14_5 to E15?"
- note removed: "This could also visually be the trace for pin 5 Which means a different location entirely"
- note removed: "maybe F12"
- note removed: "maybe F12 -> H14"
- note removed: "probably GND?"
- moved on the sheet: P1, P4, R12, R14, RN16, U_A13D, U_A14A, U_A15F, U_A1A, U_A1B, U_A2A, U_A2B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

Commit message: fix some of the interrupt lines
Connections:
- net Sys.INR0: now also P1.52 (Pin_52), RN16.6 (R5), U_A7.8 (I3a); no longer P1.49 (Pin_49), RN16.7 (R6), U_A7.6 (I2a)
- net Sys.INR1: now also P1.49 (Pin_49), RN16.7 (R6), U_A7.6 (I2a); no longer P1.50 (Pin_50), RN16.8 (R7), U_A7.4 (I1a)
- net Sys.INR2: now also P1.50 (Pin_50), RN16.8 (R7), U_A7.4 (I1a); no longer P1.51 (Pin_51), RN16.9 (R8), U_A7.2 (I0a)
- net Sys.INR3: now also P1.51 (Pin_51), RN16.9 (R8), U_A7.2 (I0a); no longer P1.52 (Pin_52), RN16.6 (R5), U_A7.8 (I3a)
- net D7A_~{S2}_Logic renamed BeginWrite
- net D7B_~{S2} renamed BeginRead
- net RENAME_MODECTL renamed DMAEnable
- net SysDataRD renamed BusCycleEnd
- no-connect marks 52 -> 54
Other:
- moved on the sheet: U_A15F, U_B11A, U_B15A, U_B15B, U_E10A, U_E11A, U_E14A, U_E14B, U_E14C, U_E14F, U_E15A, U_E15B
