File: MUX/MUX.kicad_sch (KiCad schematic)
At the start: 103 parts, among them P1 Conn_02x36_Top_Bottom, P2 DB9_Male, P3 DB9_Male, P4 DB9_Male, P5 DB9_Male

Commit message: MUX: Some annotations
Added net names for MUX0 signals and understood (and commented) function of all
writable board registers
Connections:
- net ~{CBRL}: now reaches U_E4.13 (S11), U_H7.1 (~{MR}), U_H8.1 (~{MR}), U_J5.1
- net ~{ForceTXEInt}: now reaches U_D3.9, U_E4.14 (S12)
- net RTS3_TTL: now reaches U_K8.6 (Q2), U_LL8.2
- net RTS4_TTL: now reaches U_K8.7 (Q3), U_LL8.3
- net ~{CRL1}: now reaches U_E4.1 (S0), U_E5.1
- net ~{ForceReset}: now reaches U_B6.9, U_E4.17 (S15)
- net ~{RTSL}: now reaches U_E4.9 (S8), U_E5.9
- net TXD1_BUF: now reaches U_K6.6, U_LL6.2
- net TXD1: now reaches P2.6, U_LL6.7
- net ~{TXBL4}: now reaches U_E4.8 (S7), U_H4.23 (~{TxBL})
- net ~{TXBL2}: now reaches U_E4.4 (S3), U_H2.23 (~{TxBL})
- net ~{IntEnabled}: now reaches U_D8.8 (~{Q}), U_F8.5 (EI)
- net ~{TXD1_TTL}: now reaches P2.7, U_J6.10, U_K6.5
- net ~{CRL2}: now reaches U_E4.3 (S2), U_E5.3
- net ~{TXBL3}: now reaches U_E4.6 (S5), U_H3.23 (~{TxBL})
- net RTS2: now reaches P3.4, U_L8.6
- net RTS1_TTL: now reaches U_K8.4 (Q0), U_L8.2
- net RTS2_TTL: now reaches U_K8.5 (Q1), U_L8.3
- net RTS1: now reaches P2.4, U_L8.7
- net ~{IPLL}: now reaches U_D3.13, U_E4.11 (S10)
- net ~{CRL4}: now reaches U_E4.7 (S6), U_E5.11
- net RTS_EN: now reaches U_J7.3, U_K8.14 (E)
- net ~{TXBL1}: now reaches U_E4.2 (S1), U_H1.23 (~{TxBL})
- net ~{CRL3}: now reaches U_E4.5 (S4), U_E5.5
- net CTS1: now reaches P2.2, U_L5.4 (1A)
- net RXD1: now reaches P2.8, U_L5.5 (2A)
- net TXD1_TTL: now reaches U_H1.25 (TxOUT), U_J6.11
Other:
- note added: "IPL register CP is required to load the FF ~{PE} is a shift (hi) or load (lo) signal J/K are N/C so ~{PE} must always be asserted"
- note added: "Write register address decoder"
- note removed: "CP is required to load the FF ~{PE} is a shift (hi) or load (lo) signal J/K are N/C so ~{PE} must always be asserted"
