File: MUX/MUX.kicad_sch (KiCad schematic)
At the start: 103 parts, among them P1 Conn_02x36_Top_Bottom, P2 DB9_Male, P3 DB9_Male, P4 DB9_Male, P5 DB9_Male

Commit message: some layout and labelling
Connections:
- net +5V: now also U_B8.1 (~{R}), U_B8.10 (~{S}), U_B8.13 (~{R})
- net -12V: now also U_H1.2 (NC), U_H2.2 (NC), U_H3.2 (NC), U_H4.2 (NC)
- net D4_1: now also U_B8.3 (C)
- net Data.InBD_{0}: now also U_H1.26 (TxB_{0}), U_H1.39 (EVEN/~{ODD}), U_H2.26 (TxB_{0}), U_H2.39 (EVEN/~{ODD}), U_H3.26 (TxB_{0}), U_H3.39 (EVEN/~{ODD})
- net Data.InBD_{1}: now also U_H1.27 (TxB_{1}), U_H2.27 (TxB_{1}), U_H3.27 (TxB_{1})
- net Data.InBD_{2}: now also U_H1.28 (TxB_{2}), U_H1.37 (CLS_{2}), U_H2.28 (TxB_{2}), U_H2.37 (CLS_{2}), U_H3.28 (TxB_{2}), U_H3.37 (CLS_{2})
- net Data.InBD_{3}: now also U_H1.29 (TxB_{3}), U_H1.36 (SBS), U_H2.29 (TxB_{3}), U_H2.36 (SBS), U_H3.29 (TxB_{3}), U_H3.36 (SBS)
- net Data.InBD_{4}: now also U_H1.30 (TxB_{4}), U_H1.35 (P_ENA), U_H2.30 (TxB_{4}), U_H2.35 (P_ENA), U_H3.30 (TxB_{4}), U_H3.35 (P_ENA)
- net Data.InBD_{5}: now also U_H1.31 (TxB_{5}), U_H2.31 (TxB_{5}), U_H3.31 (TxB_{5})
- net Data.InBD_{6}: now also U_H1.32 (TxB_{6}), U_H2.32 (TxB_{6}), U_H3.32 (TxB_{6})
- net Data.InBD_{7}: now also U_H1.33 (TxB_{7}), U_H2.33 (TxB_{7}), U_H3.33 (TxB_{7})
- net Data.OutD_{1}: now also U_H1.11 (RxB_{1}), U_H2.11 (RxB_{1}), U_H3.11 (RxB_{1}), U_H4.11 (RxB_{1})
- net Data.OutD_{2}: now also U_F1.5 (O2a), U_F2.5 (O2a), U_F3.5 (O2a), U_F4.5 (O2a), U_H1.10 (RxB_{2}), U_H2.10 (RxB_{2}), U_H3.10 (RxB_{2}), U_H4.10 (RxB_{2})
- net Data.OutD_{4}: now also U_F1.7 (O3a), U_F2.7 (O3a), U_F3.7 (O3a), U_F4.7 (O3a), U_H1.8 (RxB_{4}), U_H2.8 (RxB_{4}), U_H3.8 (RxB_{4}), U_H4.8 (RxB_{4})
- net Data.OutD_{5}: now also U_H1.7 (RxB_{5}), U_H2.7 (RxB_{5}), U_H3.7 (RxB_{5}), U_H4.7 (RxB_{5})
- net Data.OutD_{6}: now also U_H1.6 (RxB_{6}), U_H2.6 (RxB_{6}), U_H3.6 (RxB_{6})
- net Data.OutD_{7}: now also U_H1.5 (RxB_{7}), U_H2.5 (RxB_{7}), U_H3.5 (RxB_{7})
- net GND: now also U_B8.2 (D), U_H1.16 (~{SF_OE}), U_H2.16 (~{SF_OE}), U_H3.16 (~{SF_OE}), U_H4.16 (~{SF_OE})
- net ~{is_common_addressed}: now reaches U_B1.8, U_B6.2, U_D2.5
- net MUXClock: now reaches U_H7.2 (CP), U_H8.2 (CP), U_K1.12 (I7), U_K2.12 (I7), U_K3.12 (I7), U_K4.12 (I7), U_K5.13 (CP), U_K7.11 (Q3)
- net MUXClock: now also U_B8.11 (C)
- net INTACK: now reaches U_A7.4, U_A8.4, U_A8.5, U_C8.5
- net ~{INTACK}: now reaches U_A8.6, U_B7.12, U_C8.2
- net ~{ForceReset}: now reaches U_B6.9, U_E4.17 (S15)
- net ~{Reset}: now reaches U_A8.10, U_B7.2, U_C5.1 (~{MR}), U_D7.1, U_D7.10, U_D7.13, U_D7.4, U_D8.13 (~{R}), U_K8.15 (Clr)
- net Reset: now reaches U_A7.11, U_A8.11, U_H1.21 (RESET), U_H2.21 (RESET), U_H3.21 (RESET), U_H4.21 (RESET)
- net at U_C7.10 (CET), U_C7.9 (~{PE}), U_D2.9: no longer U_D2.4
- net at U_A7.12, U_B6.13: now also U_B8.8 (~{Q}); no longer U_B8.9 (Q)
- net ~{ReadInput}: now reaches U_B5.1 (OEa)
- net ~{ReadInput}: now also U_B5.15 (OEb)
- net D4_15 renamed ~{StatusOut}
- no-connect marks 74 -> 82
Other:
- note added: "(via)"
- note added: "-12V to support some other UART? IM6402 is NC"
- note added: "1 2 4 8 open = 1, close = 0"
- note added: "D2.8/D3.5(via)"
- note added: "rate divide by 16"
- note added: "this nand will go low when 0xF20F is accessed AND this device is interrupting AND interrupts are not preempted"
- note added: "to reset?"
- note removed: "1 2 4 8 open = 1 close = 0"
- note removed: "this nand will go low when 0xF20F is accessed AND one other condition is met (TODO)"
- note removed: "~{is common addressed}"
- moved on the sheet: JP1, JP2, JP3, JP4, R15, R_C4RN1, SW_C3, U_A1A, U_A1B, U_A1C, U_A1D, U_A1E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
