File: FFC/FFC.kicad_sch (KiCad schematic)
At the start: 226 parts, among them P1 Conn_02x36_Top_Bottom, P2 Conn_02x13_Top_Bottom, Y1 Crystal

Commit message: labels and layout on the FFC
Connections:
- net MFMClockOut: now reaches UB_B1.2, UB_E2.11 (I0b), UB_E3.12 (Q3)
- net ~{Head_Select_2^{1}}: now reaches B_P1.8 (Pin_8), B_R1.2 (R1), UB_K2.6
- net ~{Fault_Reset}: now reaches B_P1.6 (Pin_6), B_R1.3 (R2), UB_F3.10 (I4), UB_J2.6
- net ~{Direction}: now reaches B_P1.34 (Pin_34), B_R2.9 (R8), UB_F3.12 (I5), UB_K3.8
- net ~{Step}: now reaches B_P1.36 (Pin_36), B_R2.3 (R2), UB_F3.14 (I6), UB_K3.11
- net ~{Read_EN}: now reaches B_P1.4 (Pin_4), B_R1.8 (R7), UB_F3.6 (I3), UB_J2.3
- net ~{FloppyWriteData}: now reaches B_P1.38 (Pin_38), B_R3.2 (R1), UB_J2.11, UB_J2.8
- net ~{Drive_Capacity_2^{1}}: now reaches B_P1.12 (Pin_12), B_R3.3 (R2), UB_F2.6 (I2a)
- net ~{WriteProtect}: now reaches B_P1.44 (Pin_44), B_R3.7 (R6), UB_F2.17 (I3b)
- net ~{WriteFault}: now reaches B_P1.48 (Pin_48), B_R3.9 (R8), UB_F2.15 (I2b)
- net ~{DMAStartCycle}: now reaches UA_C1.8 (~{Q}), UA_C2.5, UA_L6.3
- net ~{Head_Select_2^{0}}: now reaches B_P1.14 (Pin_14), B_R1.5 (R4), UB_K3.6
- net ~{Low_Write_Current}: now reaches B_P1.2 (Pin_2), B_R1.9 (R8), UB_K2.11
- net Low_Current: now reaches UB_B3.14 (A_{4}), UB_F5.16 (Q6), UB_K2.12
- net ~{Drive_Capacity_2^{0}}: now reaches B_P1.10 (Pin_10), B_R1.4 (R3), UB_F2.4 (I1a)
- net ~{IndexPulse}: now reaches B_P1.20 (Pin_20), B_R1.7 (R6), UB_F2.11 (I0b)
- net DCR.FaultReset: now reaches UB_F6.9 (Q3), UB_J2.4, UB_J2.5
- net DCR.DriveSelect1: now reaches UB_F4.2 (IN0), UB_F6.12 (Q4), UB_J2.10
- net DCR.DriveSelect2: now reaches UB_F4.14 (IN3), UB_F6.15 (Q5)
- net DCR.DriveSelect3: now reaches UB_F4.5 (IN1), UB_F6.16 (Q6)
- net DCR.DriveSelect4: now reaches UB_F4.11 (IN2), UB_F6.19 (Q7)
- net DCR.Read_EN: now reaches UB_F6.6 (Q2), UB_J2.1, UB_J2.2
- net DMAEndCycle: now reaches UA_B1.5, UA_C2.8, UA_C3.9
- net BCtrl.~{LoadDCR1} renamed BCtrl.~{WriteDCR1}
- net BCtrl.~{LoadDCR2} renamed BCtrl.~{WriteDCR2}
- net BCtrl.~{LoadFSDR1} renamed BCtrl.~{WriteMCSR}
- net BCtrl.~{LoadFSDR23} renamed BCtrl.~{WriteFDSR12}
- net BCtrl.~{LoadSSBCH} renamed BCtrl.~{SetSSBCH}
- net BCtrl.~{LoadSSBCL} renamed BCtrl.~{SetSSBCL}
- net BCtrl.~{LoadTSM} renamed BCtrl.~{SetTSM}
- net BCtrl.~{ReadFSDR1} renamed BCtrl.~{ReadMCSR}
- net BCtrl.~{ReadFSDR2} renamed BCtrl.~{ReadFDSR1}
- net BCtrl.~{ReadFSDR3} renamed BCtrl.~{ReadFDSR2}
- net BCtrl.~{WriteFloppySync} renamed BCtrl.~{WriteFloppyPulse}
- net BStatus.Cond6 renamed BStatus.FinchDNE
- net BStatus.Cond7 renamed BStatus.MFMError
- net CardCtrl.~{RunDMA}: no longer names the net of UA_B1.2, UA_C2.3
- net Cond6 renamed FinchDNE
- net Cond7 renamed MFMError
- net Direction renamed DCR.Direction
- net FSDRSyncEN renamed MFMCheckEN
- net LoadFSDR1 renamed WriteMCSR
- net LoadFSDR2 renamed WriteFDSR1
- net Step renamed DCR.Step
- net TSMLoadDis renamed TSMSetDis
- net WriteSync renamed WritePulse
- net Write_Data_EN renamed DCR.Write_Data_EN
- net Write_Enable renamed DCR.Write_Enable
- net ~{FSDR3Clear} renamed ~{FDSR2Clear}
- net ~{FSDRSynched} renamed ~{MFMErrored}
- net ~{FSDRSync} renamed ~{ClockDataError}
- net ~{LoadCtrlReg} renamed ~{WriteCtrlReg}
- net ~{LoadDCR1} renamed ~{WriteDCR1}
- net ~{LoadDCR2} renamed ~{WriteDCR2}
- net ~{LoadFSDR1} renamed ~{WriteMCSR}
- net ~{LoadFSDR23} renamed ~{WriteFDSR12}
- net ~{LoadIPL} renamed ~{SetIPL}
- net ~{LoadIndexH} renamed ~{SetAddressH}
- net ~{LoadIndexL} renamed ~{SetAddressL}
- net ~{LoadSSBCH} renamed ~{SetSSBCH}
- net ~{LoadSSBCL} renamed ~{SetSSBCL}
- net ~{LoadTSM} renamed ~{SetTSM}
- net ~{ReadFSDR1} renamed ~{ReadMCSR}
- net ~{ReadFSDR2} renamed ~{ReadFDSR1}
- net ~{ReadFSDR3} renamed ~{ReadFDSR2}
- net ~{ReadIndexH} renamed ~{ReadAddressH}
- net ~{ReadIndexL} renamed ~{ReadAddressL}
- net ~{TSMSynched} renamed ~{TSMOutOfSync}
- net ~{WriteFloppySync} renamed ~{WriteFloppyPulse}
- net ~{Write_EN} renamed ~{Write_Enable}
Other:
- note added: "(+5V)"
- note added: "(Low Current Compensation)"
- note added: "(MFM Clock Error)"
- note added: "(N/C)"
- note added: "(half TSMClock is a ~250ns pulse)"
- note added: "3 and 2 are in a weird order!"
- note added: "C8B/C8A will only be set via ~{SetTSM} setting B8B will reset both B8B and C8A"
- note added: "Clock=0 & Data=00 & TSM_{5}=0"
- note added: "Clock=1 & Data=X1"
- note added: "MFM Clock Check"
- note added: "MFM Encoder"
- note added: "MFM/Floppy Data Registers"
- note added: "Modulation Clock Registers"
- note added: "RAM Addr H"
- note added: "RAM Addr L"
- note added: "RunDMA must be low to end the DMA request"
- note added: "either & DCR1_{b5} set"
- note added: "no end-of-cycle signal AND no cycle in progress"
- note added: "starting a cycle will request DMA"
- note added: "the A4 ROM is disabled when ~{SetTSM} is asserted"
- note removed: "(Fault Reset)"
- note removed: "(Read_EN)"
- note removed: "(TODO verify this function)"
- note removed: "(TSM Synched/Locked?)"
- note removed: "C8B/C8A will only be set via ~{LoadTSM} setting B8B will reset both B8B and C8A"
- note removed: "Low Current"
- note removed: "RAM Index H"
- note removed: "RAM Index L"
- note removed: "SYNC_{0}=0 & SDR2=0bXXXXXX00 & TSM_{5}=0"
- note removed: "SYNC_{0}=1 & SDR2=0bXXXXXXX1"
- note removed: "either & DCR1_{1} set"
- note removed: "the A4 ROM is disabled when ~{LoadTSM} is asserted"
- note removed: "~{Direction}"
- note removed: "~{Drive Capacity 2^{0}}"
- note removed: "~{Drive Capacity 2^{1}}"
- note removed: "~{Fault Reset}"
- note removed: "~{Head Select 2^{0}}"
- note removed: "~{Head Select 2^{1}}"
- note removed: "~{Low Write Current}"
- note removed: "~{Read_EN}"
- note removed: "~{Step}"
- note removed: "~{Write Data}"
- note removed: "~{Write Fault}"
- note removed: "~{Write Protect}"
- moved on the sheet: A_R10, A_R9, P2, UA_A2B, UA_A2C, UA_B1A, UA_B1C, UA_B4C, UA_C1B, UA_C2A, UA_C2B, UA_F6A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
