File: DSK/DSK.kicad_sch (KiCad schematic)
At the start: 259 parts

Commit message: DSK-I/DSK-II Card Pair WIP (mostly done)
A pair of cards connected together via a 50 pin IDC ribbon cable.
Data I/O and control for multiple CDC 9427 Hawk Drives.
Also one of the earliest Centurnion designs.
Parts:
- added BJP1: 3a/2b/1c, symbol Jumper:SolderJumper_3_Bridged12
- added BJP2: 3d/2e/1f, symbol Jumper:SolderJumper_3_Bridged12
- added B_P2: Conn_02x13_Top_Bottom, symbol Connector_Generic:Conn_02x13_Odd_Even
- added C? (x2): C_Small, symbol Device:C_Small
- added C?: C_Polarized_Small, symbol Device:C_Polarized_Small
- added D?: D_Small, symbol Device:D_Small
- added JP?: h/i, symbol Jumper:SolderJumper_2_Open
- added R? (x8): 1K, symbol Device:R
- added R?: 10K, symbol Device:R
- added R? (x2): R, symbol Device:R
- added R? (x2): ?, symbol Device:R
- added TP?: S5, symbol Connector:TestPoint
- added TP?: WG, symbol Connector:TestPoint
- added TP?: S12, symbol Connector:TestPoint
- added TP?: WAD, symbol Connector:TestPoint
- added TP?: RG, symbol Connector:TestPoint
- added TP?: S13, symbol Connector:TestPoint
- added TP?: S14, symbol Connector:TestPoint
- added TP?: DC, symbol Connector:TestPoint
- added TP?: S11, symbol Connector:TestPoint
- added TP?: S8+, symbol Connector:TestPoint
- added Y?: Crystal, symbol Device:Crystal
Connections:
- net +5V: now also UB_A7.14 (VCC), UB_B1.16 (VCC), UB_C5.14 (VCC), UB_C6.14 (VCC), UB_E6.16 (VCC), UB_E7.16 (VCC), UB_H5.16 (VCC), UB_H6.16 (VCC), UB_H7.16 (VCC), UB_J3.16 (VCC), UB_L7.16 (Vcc), R?.1, R?.1, R?.1, R?.1, R?.1, R?.1, R?.1, R?.1, R?.1, R?.1, R?.1
- net DSK2.IOAccessHigh8: now also TP?.1
- net DSK2.~{AddressError}: now also UB_F3.10, UB_H8.9 (~{Q}); no longer B_P3.39 (Pin_39), J?.39 (Pin_39), R?.1, UA_J2.9, UB_L5.3
- net DSK2.~{AddressField}: now also UB_B8.1
- net DSK2.~{CRCError}: now also UB_H8.7 (~{Q}), UB_J8.1; no longer B_P3.35 (Pin_35), J?.35 (Pin_35), R?.1, UA_J2.11, UB_L5.8
- net DSK2.~{TimeoutError}: now also UB_D6.9 (~{Q}), UB_F3.9, UB_K4.13; no longer B_P3.33 (Pin_33), J?.33 (Pin_33), R?.1, UA_J2.13, UB_L5.11
- net GND: now also UB_A7.7 (GND), UB_C5.7 (GND), UB_C6.7 (GND), UB_E6.8 (GND), UB_E7.15 (E), UB_E7.3 (I1a), UB_E7.5 (I0b), UB_E7.8 (GND), UB_F6.1, UB_F6.2, UB_H5.8 (GND), UB_H6.8 (GND), UB_H7.8 (GND), UB_J1.1 (M), UB_J1.12 (~{R}), UB_J1.15 (M), UB_J1.4 (~{R}), UB_J3.8 (GND), UB_K7.12 (D), UB_L7.8 (GND), B_P2.10 (Pin_10), B_P2.12 (Pin_12), B_P2.14 (Pin_14), B_P2.16 (Pin_16), B_P2.18 (Pin_18), B_P2.2 (Pin_2), B_P2.20 (Pin_20), B_P2.22 (Pin_22), B_P2.24 (Pin_24), B_P2.26 (Pin_26), B_P2.4 (Pin_4), B_P2.6 (Pin_6), B_P2.8 (Pin_8), C?.2, C?.2, JP?.1 (A)
- net R4.CRCError: now also UA_F3.10 (I4), UA_J2.12; no longer UA_F3.2 (I1), UA_J2.10
- net R4.TimeoutError: now also UA_F3.2 (I1), UA_J2.10; no longer UA_F3.10 (I4), UA_J2.12
- net SIn.D_{4}: now also UB_L7.13 (OUT3)
- net SIn.D_{5}: now also UB_L7.10 (OUT2)
- net SIn.D_{6}: now also UB_L7.6 (OUT1)
- net SIn.D_{7}: now also UB_L7.3 (OUT0)
- net SOut.D_{0}: now also UB_J3.12 (D2), UB_J4.13 (~{K})
- net SOut.D_{1}: now also UB_D2.12, UB_J3.13 (D3), UB_J4.14 (J)
- net SOut.D_{2}: now also UB_J3.5 (D1), UB_J4.3 (~{K})
- net SOut.D_{3}: now also UB_J3.4 (D0), UB_J4.2 (J)
- net ~{ReadState}: now also UB_L7.7 (INE)
- net ~{WriteCommand}: now also UB_D5.9; no longer UB_D5.10
- net TTL5V_K7: now reaches UB_J7.10 (~{S})
- net TTL5V_K7: now also UB_J7.1 (~{R}), UB_J7.13 (~{R}), UB_J7.4 (~{S}), UB_K7.1 (~{R}), UB_K7.13 (~{R}), UB_K7.4 (~{S}), R?.2
- net ~{HalfSelClock}: now reaches UB_J7.11 (C)
- net ~{HalfSelClock}: now also UB_K7.2 (D), UB_K7.6 (~{Q})
- net GenClockPhi1: now reaches UB_J7.12 (D)
- net GenClockPhi1: now also UB_J6.9, UB_J7.5 (Q)
- net ~{GenClock}: now reaches UB_J7.8 (~{Q})
- net ~{GenClock}: now also UB_J6.5, UB_J6.6, UB_J7.2 (D)
- net DSK1.~{Reset}: now reaches UA_B5.4, UA_F6.13 (~{MR}), UA_H2.1 (~{MR}), UA_H2.13 (~{MR}), UA_H6.13 (~{MR}), UA_H8.11 (C), UA_J1.8, UA_J6.1 (~{MR}), UA_J6.13 (~{MR})
- net WriteSR.~{CE}: now reaches UB_B5.11 (~{CE})
- net WriteSR.~{CE}: now also UB_E7.7 (Zb)
- net BitClock: now reaches UB_B5.13 (CLK)
- net BitClock: now also UB_A7.1 (A1), UB_C5.8 (CP), UB_C6.8 (CP), UB_D2.10, UB_E6.9 (Cp), UB_E7.13 (I1d), UB_E8.12 (C), UB_H5.2 (CP), UB_H6.2 (CP), UB_H7.2 (CP), UB_H8.12 (C), UB_H8.4 (C), UB_J2.12 (C), UB_K1.3, UB_K4.11
- net TTL5V_C3: now reaches UB_B4.14 (~{Clear}), UB_B5.14 (~{Clear})
- net TTL5V_C3: now also UB_B1.10 (CET), UB_C3.13 (D), UB_C4.11, R?.2
- net WriteSR.~{Load}: now reaches UB_B5.23 (SH/~{LD})
- net WriteSR.~{Load}: now also UB_E7.4 (Za)
- net ~{DMABusOE}: now reaches UB_B3.13
- net ~{DMABusOE}: now also UB_B8.3, UB_D8.1, UB_L2.6
- net ReadClock: now reaches UB_K8.5
- net ReadClock: now also UB_J1.11 (CP), UB_J5.13 (~{R}), UB_K8.4, TP?.1
- net ~{ReadClock}: now reaches UB_K8.6
- net ~{ReadClock}: now also UB_J5.1 (~{R}), UB_K7.11 (C)
- net DSK2.Busy: now reaches UB_D8.2
- net DSK2.Busy: now also UB_A7.5 (Clr), UB_B7.2, UB_E6.15 (Q3), UB_E8.15 (~{R}), UB_L4.4, UB_L4.5
- net at UB_D8.3: now also UB_D7.11
- net at UB_F1.8: now also UB_F2.1
- net CmdFormatWrite: now reaches UB_F1.9
- net CmdFormatWrite: now also UB_C4.4, UB_D4.11
- net RWData: now reaches UB_C7.1
- net RWData: now also UB_J8.8
- net CRCShiftOut: now reaches UB_C7.2
- net CRCShiftOut: now also UB_C5.13 (Q7), UB_C7.12
- net CRCShiftIn: now reaches UB_C7.3
- net CRCShiftIn: now also UB_C6.1 (DSA), UB_C6.2 (DSB), UB_C8.1
- net at UB_J8.11: now also UB_J8.10
- net WriteData: now reaches UB_J8.12
- net WriteData: now also UB_C7.5, UB_E3.10 (~{Y}), UB_J6.8
- net DSK2.~{ReadGate}: now reaches UB_J8.13
- net DSK2.~{ReadGate}: now also UB_F5.6, UB_K4.4
- net at UB_D7.5: now also UB_D8.6
- net SMStart: now reaches UB_D7.6, UB_F4.8 (D_{0})
- net at UB_K4.10: now also UB_K3.13, UB_K3.4
- net DSK.~{INTStrobe}: now reaches J?.31 (Pin_31), UA_K3.3
- net DSK.~{INTStrobe}: now also B_P3.31 (Pin_31), R?.2, UB_K6.9
- net DSK.~{Reset}: now reaches J?.45 (Pin_45), R?.1, UA_J1.11
- net DSK.~{Reset}: now also B_P3.45 (Pin_45), UB_L4.8
- net DSK.~{CmdSeek}: now reaches J?.49 (Pin_49), R?.1, UA_K1.1 (A), UA_K1.10 (B)
- net DSK.~{CmdSeek}: now also B_P3.49 (Pin_49), UB_L4.3
- net ReadData: now reaches UB_C7.10
- net ReadData: now also UB_B4.1 (~{K}), UB_B4.2 (J), UB_C7.4, UB_H3.3 (I1a), UB_H3.6 (I1b), UB_J8.4, UB_K7.9 (Q)
- net ~{AddrReadEqual}: now reaches UB_C7.8
- net ~{AddrReadEqual}: now also UB_B7.9
- net at UB_C7.9: now also UB_B8.2
- net at UB_F8.10 (~{S}): now also UB_C8.10, UB_D8.11
- net ~{DMAReadReady}: now reaches UB_F8.11 (C)
- net ~{DMAReadReady}: now also UB_E7.14 (I0d), UB_L3.6
- net TTL5V_F8: now reaches UB_F8.12 (D)
- net TTL5V_F8: now also UB_E6.1 (~{Mr}), UB_E8.11 (~{S}), UB_E8.2 (J), UB_E8.3 (~{K}), UB_E8.5 (~{S}), UB_F6.11, UB_F6.3, UB_F8.2 (D), UB_F8.4 (~{S}), R?.2
- net ~{NeedLoadByte}: now reaches UB_F8.13 (~{R})
- net ~{NeedLoadByte}: now also UB_E7.2 (I0a), UB_F6.8
- net at UB_F8.9 (Q): now also UB_D7.9
- net at UB_K1.10: now also UB_K1.6, UB_K1.9, R?.1, R?.2
- net at UB_K1.8: now also UB_K1.12, UB_K1.13, R?.2, Y?.2
- net at UB_F2.4: now also UB_F1.11
- net at UB_F2.5: now also UB_F1.6
- net DSK2.ReadGate: now reaches UB_F2.6
- net DSK2.ReadGate: now also UB_H3.1 (S), UB_J8.5, UB_K4.3, UB_L7.11 (IN2), TP?.1
- net TTL5V_D6: now reaches UB_D6.11 (~{S})
- net TTL5V_D6: now also UB_D6.13 (~{K}), UB_D6.3 (~{K}), UB_D6.5 (~{S}), R?.2
- net GenClock: now reaches UB_D6.12 (C)
- net GenClock: now also UB_D6.4 (C), UB_E4.11 (C), UB_H3.14 (I0d), UB_J1.5 (CP), UB_J5.11 (C), UB_J5.3 (C), UB_J6.4
- net at UB_D6.14 (J): now also UB_D7.2
- net ~{ClearErrors}: now reaches UB_D6.15 (~{R})
- net ~{ClearErrors}: now also UB_D6.1 (~{R}), UB_H8.1 (~{R}), UB_H8.15 (~{R}), UB_J2.1 (~{R}), UB_J2.15 (~{R}), UB_J6.1
- net CmdFormatWriteDo: now reaches UB_C3.10 (Q5)
- net CmdFormatWriteDo: now also UB_D4.13
- net CmdFormatWriteInit: now reaches UB_C3.11 (Q6)
- net CmdFormatWriteInit: now also UB_D4.12
- net CmdSM_A_{4}: now reaches UB_A1.5 (D1), UB_C3.12 (Q7)
- net ~{EndCommand}: now reaches UB_C3.15 (Clr), UB_D3.12, UB_D5.5
- net CmdRead: now reaches UB_C3.4 (Q0)
- net CmdRead: now also UB_B4.23 (SH/~{LD}), UB_C4.1, UB_D2.5, UB_D3.5, UB_E7.1 (S)
- net CmdWrite: now reaches UB_C3.5 (Q1)
- net CmdWrite: now also UB_C4.2, UB_F1.12, UB_F1.2
- net CmdSeek: now reaches UB_C3.6 (Q2)
- net CmdSeek: now also UB_D2.2, UB_L4.1, UB_L4.2
- net CmdVerify: now reaches UB_C3.9 (Q4), UB_C4.5, UB_D2.4
- net CmdVerify: now also UB_F7.10
- net at UB_F2.2: now also UB_F1.3
- net SMWriteGate: now reaches UB_F2.3
- net SMWriteGate: now also UB_K2.2, TP?.1
- net at UB_C1.10 (~{S}): now also UB_D7.4
- net DSK2.INTStrobe: now reaches UB_C1.11 (C)
- net DSK2.INTStrobe: now also UB_K6.8
- net InterruptRequest: now reaches UB_C1.8 (~{Q})
- net InterruptRequest: now also UB_K2.13
- net at UB_L1.4: now also UB_K2.11
- net at UB_L1.5: now also UB_K2.10, UB_L1.10, UB_L1.12, UB_L3.2
- net DMA.~{INTRequest}: now reaches UB_L1.6
- net DMA.~{INTRequest}: now also B_P2.23 (Pin_23)
- net at UB_L2.1: now also UB_J5.5 (Q)
- net at UB_L2.2: now also UB_J5.9 (Q)
- net at UB_L2.3: now also UB_K2.4
- net DiagSectorPulse: now reaches UB_L8.1
- net DiagSectorPulse: now also UB_J3.15 (Q3)
- net DiagEnable: now reaches UB_L8.2
- net DiagEnable: now also UB_A7.2 (A2), UB_D7.13, UB_J3.2 (Q0), UB_K5.12, UB_K5.4, UB_L8.10, UB_L8.4
- net ~{EndOfDMA}: now reaches UB_J8.2
- net ~{EndOfDMA}: now also UB_B7.4, UB_D8.10, UB_K2.8, UB_L1.2
- net at UB_J8.3: now also UB_K3.1, UB_L3.3
- net at UB_K1.1: now also UB_J1.7 (~{Y})
- net at UB_K1.2: now also UB_J1.9 (~{Y})
- net ~{DiagEnable}: now reaches UB_D7.12
- net ~{DiagEnable}: now also UB_D5.13
- net TTL5V_4: now reaches R?.2, UA_E8.10 (~{S}), UA_E8.12 (D), UA_E8.2 (D), UA_E8.4 (~{S}), UA_F8.10 (~{S}), UA_F8.12 (D), UA_F8.2 (D), UA_F8.4 (~{S}), UA_H8.1 (~{R}), UA_H8.4 (~{S})
- net at UB_K3.10: now also BJP1.2 (C)
- net at UB_K3.11: now also UB_L3.8
- net at UB_K3.8: now also UB_L2.10, UB_L2.13, UB_L2.4, UB_L3.1
- net at UB_K3.9: now also BJP2.2 (C)
- net State10ReadVerify: now reaches UB_C8.2
- net State10ReadVerify: now also UB_F5.10
- net at UB_C8.3: now also UB_C8.4
- net DiagClock: now reaches UB_K5.5
- net DiagClock: now also UB_J4.10 (Q)
- net ~{OCSelClock}: now reaches UB_K5.6
- net ~{OCSelClock}: now also UB_K4.9, UB_K5.8, R?.2
- net ~{EndSeekCommand}: now reaches UB_D3.4
- net ~{EndSeekCommand}: now also UB_F7.13
- net HalfSelClock: now reaches UB_J7.3 (C)
- net HalfSelClock: now also UB_J6.12, UB_K7.5 (Q)
- net DSK2.CRCError: now reaches UB_L5.12, UB_L5.13
- net DSK2.CRCError: now also UB_H8.6 (Q)
- net DMA.~{BusWriteOE}: now reaches UB_L2.5
- net DMA.~{BusWriteOE}: now also B_P2.17 (Pin_17)
- net at UB_L2.8: now also UB_L3.5
- net DMA.~{BusReadReady}: now reaches UB_L2.9
- net DMA.~{BusReadReady}: now also B_P2.15 (Pin_15)
- net SetCRCError: now reaches UB_H8.2 (J)
- net SetCRCError: now also UB_C8.6
- net TTL5V_H7: now reaches UB_H8.3 (~{K})
- net TTL5V_H7: now also UB_H3.13 (I1d), UB_H5.1 (~{MR}), UB_H6.1 (~{MR}), UB_H7.1 (~{MR}), UB_H7.10 (CET), UB_H7.7 (CEP), UB_H8.11 (~{S}), UB_H8.13 (~{K}), UB_H8.5 (~{S}), R?.2
- net at UB_F4.1 (D_{7}): now also UB_H3.4 (Za)
- net ~{SMAdvance}: now reaches UB_E3.1 (D_{7}), UB_E3.16 (D_{15}), UB_F4.10 (~{Y}), UB_F5.12, UB_H5.9 (~{PE})
- net ~{SMAdvance}: now also UB_D2.9, UB_F5.3, UB_H6.9 (~{PE}), UB_H7.9 (~{PE})
- net at UB_F4.16 (D_{15}): now also UB_H3.7 (Zb)
- net at UB_F4.17 (D_{14}): now also UB_K8.12
- net BitIndex_{5}: now reaches UB_F4.18 (D_{13}), UB_F4.19 (D_{12}), UB_F4.4 (D_{4}), UB_F4.6 (D_{2})
- net BitIndex_{5}: now also UB_H6.13 (Q1)
- net BitIndex_{7}: now reaches UB_F4.2 (D_{6}), UB_F4.5 (D_{3}), UB_F4.7 (D_{1}), UB_H3.2 (I0a)
- net BitIndex_{7}: now also UB_H6.11 (Q3)
- net WordIndex: now reaches UB_F4.20 (D_{11})
- net WordIndex: now also UB_F4.21 (D_{10}), UB_F4.22 (D_{9}), UB_F4.3 (D_{5}), UB_H5.7 (CEP), UB_H6.7 (CEP), UB_H7.15 (TC), UB_K5.2
- net at UB_L1.1: now also UB_E8.10 (Q)
- net DMA.~{Request}: now reaches UB_L1.3
- net DMA.~{Request}: now also B_P2.25 (Pin_25)
- net State.S8: now reaches UB_K3.3
- net State.S8: now also UB_H1.6, UB_K3.2, TP?.1
- net at UB_K3.5: now also UB_L3.4
- net DSK2.~{SectorAddressInc}: now reaches UB_K3.6
- net DSK2.~{SectorAddressInc}: now also UB_E8.13 (~{K}), UB_K4.5
- net State.~{S9}: now reaches TP?.1, UB_H2.10 (S9)
- net State.S7: now reaches UB_H1.10
- net State.S7: now also UB_F2.13
- net State.~{S7}: now reaches UB_H1.11
- net State.~{S7}: now also TP?.1, UB_D8.12, UB_F5.11, UB_H2.8 (S7)
- net at UB_D3.13: now also UB_F7.12
- net DSK2.~{SepReadData}: now reaches UB_K7.10 (~{S})
- net DSK2.~{SepReadData}: now also UB_K8.8
- net ~{State14VerifyDataFail}: now reaches UB_C8.5
- net ~{State14VerifyDataFail}: now also UB_F7.8
- net ~{SysDataOut}: now reaches UB_A4.9 (OE)
- net ~{SysDataOut}: now also UB_A5.9 (OE), UB_D4.8
- net ~{SMReset}: now reaches UB_F7.1
- net ~{SMReset}: now also UB_C4.8, UB_E2.1 (~{MR})
- net at UB_F7.2: now also UB_K3.12
- net ~{CRCShiftOut}: now reaches UB_C7.11
- net ~{CRCShiftOut}: now also UB_E3.21 (D_{10})
- net at UB_C7.13: now also JP?.2 (B), R?.2
- net at UB_E8.1 (~{R}): now also UB_D7.10
- net at UB_E8.4 (C): now also UB_D8.8
- net at UB_E8.6 (Q): now also UB_E7.10 (I1c)
- net at UB_F6.10: now also UB_E6.5 (D1), UB_F6.6, UB_F6.9, C?.1
- net at UB_F6.12: now also UB_E8.14 (J), UB_F5.13
- net at UB_F6.13: now also UB_F5.1
- net DSK2.~{Reset}: now reaches UB_B1.1 (~{MR}), UB_B3.11, UB_D3.9, UB_D4.6, UB_J3.1 (~{Mr})
- net DSK2.~{Reset}: now also UB_D5.10
- net at UB_B1.2 (CP): now also UB_A1.9 (Cp), UB_A2.8
- net at UB_A1.1 (~{Mr}), UB_B1.7 (CEP): now also UB_A1.14 (~{Q3})
- net AnySeekCommand: now reaches UB_B1.9 (~{PE})
- net AnySeekCommand: now also UB_D2.3
- net BusyFlag: now reaches UB_D5.4
- net BusyFlag: now also UB_D5.3, UB_E6.13 (D3)
- net at UB_D5.6: now also UB_D5.2
- net at UB_F2.11: now also UB_F3.3
- net BitIndex_{8}: now reaches UB_F2.12
- net BitIndex_{8}: now also UB_H5.14 (Q0)
- net ~{DSK2IORead}: now reaches UB_B2.12 (A3), UB_D1.8, UB_D4.9
- net DSK2.Reset: now reaches UB_D3.8
- net DSK2.Reset: now also UB_C1.3 (C), UB_C4.10, UB_C4.9, UB_L4.10, UB_L4.9
- net State.~{S10}: now reaches TP?.1, UB_H2.11 (S10)
- net State.~{S10}: now also UB_F5.8
- net BitIndex_{2}: now reaches UB_H6.10 (CET)
- net BitIndex_{2}: now also UB_F7.4, UB_H7.12 (Q2), UB_L6.1, UB_L6.2
- net BitIndex_{4}: now reaches UB_H6.14 (Q0)
- net BitIndex_{4}: now also UB_F2.9
- net at UB_H6.15 (TC): now also UB_H5.10 (CET)
- net at UB_H6.6 (D3): now also UB_H1.2, UB_H5.3 (D0), UB_H5.4 (D1)
- net EndSyncWait: now reaches UB_H1.9, UB_J1.3 (~{S2})
- net EndSyncWait: now also UB_H4.15 (TC), UB_K2.5
- net TTL5V_J5: now reaches UB_J4.11 (~{S})
- net TTL5V_J5: now also UB_H4.10 (CET), UB_H4.9 (~{PE}), UB_J4.1 (~{R}), UB_J4.15 (~{R}), UB_J4.5 (~{S}), UB_J5.10 (~{S}), UB_J5.12 (D), UB_J5.2 (D), UB_J5.4 (~{S}), R?.2
- net ~{WriteDiagClocks}: now reaches UB_J4.12 (C)
- net ~{WriteDiagClocks}: now also UB_C2.3 (2), UB_J4.4 (C)
- net ~{BadPreemble}: now reaches UB_F3.1
- net ~{BadPreemble}: now also UB_J2.9 (~{Q})
- net DSK2.FormatError: now reaches UB_F3.12
- net DSK2.FormatError: now also UB_K4.1, UB_L5.4, UB_L5.5
- net ~{ReadClockFail}: now reaches UB_F3.13
- net ~{ReadClockFail}: now also UB_D6.7 (~{Q})
- net ~{UnexpectedSector}: now reaches UB_F3.2
- net ~{UnexpectedSector}: now also UB_J2.7 (~{Q})
- net DiagOnSector: now reaches UB_K5.13
- net DiagOnSector: now also UB_J3.7 (Q1)
- net SectorPulse: now reaches UB_K8.2
- net SectorPulse: now also UB_F8.3 (C), UB_J2.4 (C)
- net State.S5Read: now reaches UB_F5.4
- net State.S5Read: now also UB_B7.10
- net State.~{S5}: now reaches UB_F5.5
- net State.~{S5}: now also UB_H2.6 (S5), TP?.1
- net at UB_A1.13 (D3): now also UB_A1.2 (Q0)
- net at UB_A1.4 (D0): now also UB_A2.12
- net INTStrobe: now reaches UA_H8.5 (Q), UA_K3.1, UA_K3.2
- net at UB_D1.1, UB_D3.2: no longer UB_A3.2
- net at UB_B7.5: now also UB_B8.8
- net at UB_B7.6: now also UB_B8.11
- net at UB_L3.12: now also BJP2.3 (B)
- net DMA.~{Control0}: now reaches UB_L3.13
- net DMA.~{Control0}: now also BJP2.1 (A), B_P2.5 (Pin_5)
- net State.~{S6}: now reaches TP?.1, UB_H2.7 (S6)
- net PreembleFormatError: now reaches UB_H3.10 (I1c)
- net PreembleFormatError: now also UB_F3.6
- net BitIndex_{3}: now reaches UB_H3.5 (I0b)
- net BitIndex_{3}: now also UB_H7.11 (Q3), UB_L6.12, UB_L6.13
- net ReadFormatError: now reaches UB_H3.9 (Zc)
- net ReadFormatError: now also UB_J2.14 (J)
- net TTL5V_J2: now reaches UB_J2.11 (~{S})
- net TTL5V_J2: now also R?.2, UB_J2.13 (~{K}), UB_J2.3 (~{K}), UB_J2.5 (~{S})
- net State.S15: now reaches TP?.1, UB_H1.12
- net State.S15: now also UB_F2.10
- net State.~{S15}: now reaches UB_H1.13, UB_H2.17 (S15)
- net DSK2.ReadyOnSector: now reaches UB_K6.2
- net DSK2.ReadyOnSector: now also UB_C4.3, UB_K6.13
- net at UB_J6.10: now also UB_J6.11
- net BitIndex_{1}: now reaches UB_F7.3
- net BitIndex_{1}: now also UB_H7.13 (Q1), UB_L6.4, UB_L6.5
- net BitIndex_{0}: now reaches UB_F7.5
- net BitIndex_{0}: now also UB_H4.2 (CP), UB_H7.14 (Q0), UB_L6.10, UB_L6.9
- net ~{ByteIndex}: now reaches UB_F7.6
- net ~{ByteIndex}: now also UB_F6.5
- net State.~{S0}: now reaches TP?.1, UB_H2.1 (S0), UB_J2.2 (J)
- net DiagReadDataLoopback: now reaches UB_J3.10 (Q2)
- net DiagReadDataLoopback: now also UB_L8.9
- net DiagDisabled: now reaches UB_J3.3 (~{Q0})
- net DiagDisabled: now also UB_K5.10
- net ~{WriteDiag9}: now reaches UB_J3.9 (Cp)
- net ~{WriteDiag9}: now also UB_C2.2 (1)
- net at UB_L5.10, UB_L5.9: now also UB_K4.12
- net at UB_B8.5: now also UB_B7.8
- net SetAddressError: now reaches UB_B8.6
- net SetAddressError: now also UB_H8.14 (J)
- net at UB_B7.1: now also UB_A7.6 (~{Q})
- net at UB_B7.3: now also UB_D7.1
- net State.N_{3}: now reaches UB_A3.9, UB_D1.2, UB_E1.4 (Q_{3}), UB_E2.4 (P0)
- net ~{SoftReset}: now reaches UB_C2.4 (3), UB_D4.5
- net ~{NextState14}: now reaches UB_D1.6, UB_H1.1
- net ~{NextState14}: now also UB_C5.9 (~{MR}), UB_C6.9 (~{MR}), UB_F5.2
- net InterruptsOn: now reaches UB_C1.5 (Q)
- net InterruptsOn: now also UB_K2.12
- net at UB_J4.6 (Q): now also UB_L8.5
- net DSK2.WriteAllow: now reaches UB_K2.1
- net DSK2.WriteAllow: now also UB_K6.4
- net DSK2.WriteGate: now reaches UB_K2.3
- net DSK2.WriteGate: now also UB_D4.2, UB_L7.2 (IN0), UB_L7.5 (IN1)
- net at UB_B8.4: now also UB_D5.12
- net at UB_H1.8, UB_J1.14 (~{S2}): now also UB_H4.7 (CEP); no longer UB_H4.2 (CP)
- net StartOfSectorBit: now reaches UB_E6.10 (Q2)
- net StartOfSectorBit: now also UB_D8.5
- net ~{StartOfSectorBit}: now reaches UB_E6.11 (~{Q2})
- net ~{StartOfSectorBit}: now also UB_F8.1 (~{R})
- net StartOfSector: now reaches UB_E6.12 (D2)
- net StartOfSector: now also UB_F8.5 (Q)
- net SMCommand: now reaches UB_E6.3 (~{Q0})
- net SMCommand: now also UB_D8.4
- net ~{SMCommand}: now reaches UB_E6.4 (D0)
- net ~{SMCommand}: now also UB_C4.6
- net at UB_E6.6 (~{Q1}): now also UB_E7.6 (I1b)
- net at UB_E6.7 (Q1): now also UB_D8.9
- net State.~{S14}: now reaches UB_H1.3
- net State.~{S14}: now also UB_F6.4, UB_H2.16 (S14), TP?.1
- net State.S14: now reaches UB_H1.4
- net State.S14: now also UB_F7.9
- net State.N_{2}: now reaches UB_A3.12, UB_D1.4, UB_E1.3 (Q_{2}), UB_E2.5 (P1)
- net State.N_{1}: now reaches UB_A3.5, UB_D1.5, UB_E1.2 (Q_{1}), UB_E2.6 (P2)
- net State.~{S4}: now reaches TP?.1, UB_H2.5 (S4)
- net at UB_J8.9: now also UB_J8.6
- net DMA.~{EndOfBuffer}: now reaches UB_K2.9
- net DMA.~{EndOfBuffer}: now also B_P2.9 (Pin_9)
- net SelClock: now reaches UB_K4.8
- net SelClock: now also UB_K7.3 (C)
- net SetReadClockFail: now reaches UB_K2.6
- net SetReadClockFail: now also UB_D6.2 (J)
- net CrystalClock: now reaches UB_K1.11
- net CrystalClock: now also UB_K5.9
- net WriteDataCom: now reaches UB_D4.1
- net WriteDataCom: now also UB_J6.13
- net GateWriteDataCom: now reaches UB_D4.3
- net GateWriteDataCom: now also UB_L7.14 (IN3)
- net CmdsReadVerify: now reaches UB_C8.12, UB_C8.13, UB_D2.6, UB_F1.5
- net at UB_D3.6: now also UB_L1.9
- net ~{RWDataEqual}: now reaches UB_F7.11
- net ~{RWDataEqual}: now also UB_C7.6
- net at UB_K8.10: now also UB_K8.9
- net ~{SepReadData}: now reaches UB_K8.11
- net ~{SepReadData}: now also B_P3.1 (Pin_1), J?.1 (Pin_1), J?.42, R?.2, UB_L8.8
- net DMA.~{Enable}: now reaches UB_L3.9
- net DMA.~{Enable}: now also B_P2.11 (Pin_11)
- net at UB_F3.4: now also UB_F2.8, UB_F3.5
- net at UB_C8.8: now also UB_D8.13
- net at UB_C8.9: now also UB_B8.10
- net at UB_D5.8: now also UB_J6.2, UB_J6.3
- net CRCShift8: now reaches UB_C6.13 (Q7)
- net CRCShift8: now also UB_C5.1 (DSA), UB_C5.2 (DSB)
- net at UB_K1.4: now also UB_K1.5, R?.1, Y?.1
- net State.~{S11}: now reaches UB_H2.13 (S11)
- net State.~{S11}: now also TP?.1
- net State.~{S12}: now reaches UB_H2.14 (S12)
- net State.~{S12}: now also TP?.1
- net State.~{S13}: now reaches UB_H2.15 (S13)
- net State.~{S13}: now also TP?.1
- net State.~{S1}: now reaches TP?.1, UB_H2.2 (S1)
- net State.~{S2}: now reaches TP?.1, UB_H2.3 (S2)
- net State.~{S3}: now reaches TP?.1, UB_H2.4 (S3)
- net State.~{S8}: now reaches UB_H2.9 (S8)
- net State.~{S8}: now also UB_H1.5
- net ~{CmdsReadVerify}: now reaches UB_F5.9
- net ~{CmdsReadVerify}: now also UB_C8.11
- net DSK2.AddressError: now reaches UB_L5.1, UB_L5.2
- net DSK2.AddressError: now also UB_H8.10 (Q)
- net at UB_K8.13: now also UB_K5.3, R?.2
- net at UB_D5.11: now also UB_D4.10
- net at UB_K4.2: now also UB_F3.11
- net at UB_E7.11 (I0c): now also UB_D7.8
- net ReadSRClock: now reaches UB_E7.12 (Zd)
- net ReadSRClock: now also UB_B4.11 (~{CE}), UB_B4.13 (CLK)
- net DMAStartCycle: now reaches UB_E7.9 (Zc)
- net DMAStartCycle: now also UB_L1.13
- net at UB_K4.6: now also UB_L4.12, UB_L4.13
- net ~{GateOE}: now reaches UB_L7.9 (OE)
- net ~{GateOE}: now also UB_K6.12
- net at UB_C4.12: now also UB_C4.13, UB_E4.9 (Q)
- net at UB_A7.11 (Cext): now also C?.2
- net at UB_A7.13 (R/Cext): now also D?.1 (K)
- net at UB_A7.3 (B1): now also UB_A7.4 (B2), R?.2
- net ~{ClearInterrupt}: now reaches UB_C2.9 (7)
- net ~{ClearInterrupt}: now also UB_B3.9
- net at UB_E4.12 (D): now also UB_E4.5 (Q)
- net at UB_E4.8 (~{Q}): now also UB_E4.1 (~{R})
- net EndBlock: now reaches UB_K5.1
- net EndBlock: now also UB_B8.9, UB_H5.15 (TC), C?.1
- net State.N_{0}: now reaches UB_D3.1, UB_E1.1 (Q_{0}), UB_E2.7 (P3)
- net State.N_{0}: now also UB_A3.2
- net at UB_D7.3: now also UB_B3.8
- net at UB_E4.3 (C): now also UB_F3.8
- net DMA.Write/~{Read}: now reaches UB_L1.8
- net DMA.Write/~{Read}: now also B_P2.21 (Pin_21)
- net DMA.~{StartCycle}: now reaches UB_L1.11
- net DMA.~{StartCycle}: now also B_P2.19 (Pin_19)
- net ~{DMAINTAcknowledge}: now reaches UB_B3.10
- net ~{DMAINTAcknowledge}: now also UB_L2.11
- net DMA.~{INTAcknowledge}: now reaches UB_L2.12
- net DMA.~{INTAcknowledge}: now also B_P2.13 (Pin_13)
- net at UB_L3.10: now also BJP1.3 (B)
- net DMA.~{Control1}: now reaches UB_L3.11
- net DMA.~{Control1}: now also BJP1.1 (A), B_P2.7 (Pin_7)
- net DSK.AssertAddress renamed DSK1.AssertAddress
- net DSK.Busy renamed DSK1.Busy
- net DSK.~{Protected} renamed DSK1.~{Protected}
- net DSK2.AddressFieldBit renamed DSK.AddressFieldBit
- net DSK2.RTZSeek renamed CmdRTZSeek
- net DSK2.SectorAddressInc renamed DSK.SectorAddressInc
- net DSK2.~{AFA_{0}} renamed DSK.~{AFA_{0}}
- net DSK2.~{AFA_{1}} renamed DSK.~{AFA_{1}}
- net DSK2.~{AFA_{2}} renamed DSK.~{AFA_{2}}
- net DSK2.~{AFA_{3}} renamed DSK.~{AFA_{3}}
- net DSK2.~{Busy} renamed DSK.~{Busy}
- net DSK2.~{FormatError} renamed DSK.~{FormatError}
- net DSK2.~{IOAccessHigh8} renamed DSK.~{IOAccessHigh8}
- net DSK2.~{ReadyOnSector} renamed DSK.~{ReadyOnSector}
- net DSK2.~{WriteAllow} renamed DSK.~{WriteAllow}
- net StateA_{0} renamed State.A_{0}
- net StateA_{1} renamed State.A_{1}
- net StateA_{2} renamed State.A_{2}
- net StateA_{3} renamed State.A_{3}
- net ~{DSK.Busy} renamed ~{DSK1.Busy}
- net ~{SepClock} renamed ~{SepReadClock}
- removed net ~{SepData}: B_P3.1 (Pin_1), J?.1 (Pin_1), J?.42, R?.2, UB_K8.9, UB_L8.8
- net ~{WriteData} renamed ~{CombWriteData}
- new net: C?.1, D?.2 (A), R?.2
- new net DSK.~{AddressError}: B_P3.39 (Pin_39), J?.39 (Pin_39), R?.1, UA_J2.9, UB_L5.3
- new net DSK.~{CRCError}: B_P3.33 (Pin_33), J?.33 (Pin_33), R?.1, UA_J2.13, UB_L5.11
- new net DSK.~{TimeoutError}: B_P3.35 (Pin_35), J?.35 (Pin_35), R?.1, UA_J2.11, UB_L5.8
- no-connect marks 107 -> 162
Other:
- note added: "+WriteData"
- note added: "0"
- note added: "1"
- note added: "2"
- note added: "3"
- note added: "Busy Enables on: Read/Write/Verify/Format"
- note added: "Busy clearing OR any Hawk Interrupt line asserting"
- note added: "Control Enable"
- note added: "DMA.~{AddressControl}"
- note added: "DSK Read will Write to DMA Other Commands Read from DMA"
- note added: "GenClock"
- note added: "H7 will increment the H6/H5 pair every 16 bits. If entering state 14, H6/H5 will load with 0x38. Terminal count will happen after 3200 (0xC80) bits, or 400 (0x190) Bytes. Other states load 0, and Terminal count after 4096 bits."
- note added: "Key Pin"
- note added: "Not used on CPU6"
- note added: "Reading 128 Bits in State 7 OR 16 Bits in State 15 Triggers FormatError"
- note added: "SectorPulse while not waiting for sector is a FormatError"
- note added: "SelClock"
- note added: "When ReadGate turns on This will wait 29 GenClock times then switch to ReadClock."
- note added: "WriteDataCom"
- moved on the sheet: R?, TP?, UA_D2A, UA_D2B, UA_J4A, UA_J4B, UB_A1, UB_A2D, UB_A2E, UB_A2F, UB_A3A, UB_A3B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
