File: DSK/DSK.kicad_sch (KiCad schematic)
At the start: 291 parts, among them Y1 10MHz

Commit message: misc readability, fix MUX errata
Other:
- note added: "Reading 256 Bits in State 7 OR 16 Bits in State 15 Triggers FormatError"
- note removed: "Reading 128 Bits in State 7 OR 16 Bits in State 15 Triggers FormatError"
Changed lines of the file:
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@@
     (effects (font (size 1.27 1.27)) (justify right bottom))
   )
-  (text "Reading 128 Bits in State 7\nOR 16 Bits in State 15\nTriggers FormatError"
+  (text "Reading 256 Bits in State 7\nOR 16 Bits in State 15\nTriggers FormatError"
     (at 739.14 933.45 0)
     (effects (font (size 1.27 1.27)) (justify left bottom))
